File: schematic.sch (EAGLE design)
At the start: 0 parts

Commit message: Added ATSAM3S2CA-AU to the schematic.
Parts:
- added U1: ATSAM3S2CA-AU, Atmel_By_element14_Batch_1-00:ATSAM3S2CA-AU
Changed lines of the file:
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@@
 </classes>
 <parts>
+<part name="U1" library="Atmel_By_element14_Batch_1-00" deviceset="ATSAM3S2CA-AU" device=""/>
 </parts>
 <sheets>
@@
 </plain>
 <instances>
+<instance part="U1" gate="A" x="116.84" y="101.6"/>
 </instances>
 <busses>

Commit message: added a schemetic symbol for the FTDI chip.
Connections:
- new net GND: U1.GND, U1.GND_2, U1.GND_3, U1.GND_4, U1.GND_5
Changed lines of the file:
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@@
 <?xml version="1.0" encoding="utf-8"?>
 <!DOCTYPE eagle SYSTEM "eagle.dtd">
-<eagle version="7.4.0">
+<eagle version="7.3.0">
 <drawing>
 <settings>
@@
 <parts>
 <part name="U1" library="Atmel_By_element14_Batch_1-00" deviceset="ATSAM3S2CA-AU" device=""/>
+<part name="SUPPLY1" library="supply2" deviceset="GND" device=""/>
 </parts>
 <sheets>
@@
 <instances>
 <instance part="U1" gate="A" x="116.84" y="101.6"/>
+<instance part="SUPPLY1" gate="GND" x="81.28" y="20.32"/>
 </instances>
 <busses>
 </busses>
 <nets>
+<net name="GND" class="0">
+<segment>
+<pinref part="U1" gate="A" pin="GND_2"/>
+<wire x1="86.36" y1="38.1" x2="81.28" y2="38.1" width="0.1524" layer="91"/>
+<wire x1="81.28" y1="38.1" x2="81.28" y2="35.56" width="0.1524" layer="91"/>
+<pinref part="U1" gate="A" pin="GND_3"/>
+<wire x1="81.28" y1="35.56" x2="86.36" y2="35.56" width="0.1524" layer="91"/>
+<wire x1="81.28" y1="35.56" x2="81.28" y2="33.02" width="0.1524" layer="91"/>
+<junction x="81.28" y="35.56"/>
+<pinref part="U1" gate="A" pin="GND_4"/>
+<wire x1="81.28" y1="33.02" x2="86.36" y2="33.02" width="0.1524" layer="91"/>
+<wire x1="81.28" y1="33.02" x2="81.28" y2="30.48" width="0.1524" layer="91"/>
+<junction x="81.28" y="33.02"/>
+<pinref part="U1" gate="A" pin="GND_5"/>
+<wire x1="81.28" y1="30.48" x2="81.28" y2="27.94" width="0.1524" layer="91"/>
+<wire x1="81.28" y1="27.94" x2="81.28" y2="22.86" width="0.1524" layer="91"/>
+<wire x1="86.36" y1="30.48" x2="81.28" y2="30.48" width="0.1524" layer="91"/>
+<junction x="81.28" y="30.48"/>
+<pinref part="U1" gate="A" pin="GND"/>
+<wire x1="86.36" y1="27.94" x2="81.28" y2="27.94" width="0.1524" layer="91"/>
+<junction x="81.28" y="27.94"/>
+<pinref part="SUPPLY1" gate="GND" pin="GND"/>
+</segment>
+</net>
 </nets>
 </sheet>
