File: schematic/schematic.sch (EAGLE design)
At the start: 68 parts, among them U1 ATSAM3S2CA-AU

Commit message: Finished up the current FTDI and iCE connection
Parts:
- added C35, C37, C39: 0.1uF, resistor:C-USC0805
- added C36, C38: 4.7uF, resistor:C-USC0805
- added C40: 10uF, resistor:C-USC0805
- added R28: 2.2K, resistor:R-US_M1206
- added R29: 12K, resistor:R-US_M1206
- added R30, R31, R32, R33, R34, R35, R36: 0, resistor:R-US_M1206
Connections:
- new net CTSN: R33.1
- new net DCDN: R36.1
- new net DSRN: R35.1
- new net DTRN: R34.1
- new net N$19: R28.1, U$1.!RESET
- new net N$20: R29.1, U$1.REF
- new net N$23: C39.2, C40.2, R29.2
- new net N$24: R30.2, U$1.BDBUS0
- new net N$25: R31.2, U$1.BDBUS1
- new net N$26: R32.2, U$1.BDBUS2
- new net N$27: R33.2, U$1.BDBUS3
- new net N$28: R34.2, U$1.BDBUS4
- new net N$29: R35.2, U$1.BDBUS5
- new net N$30: R36.2, U$1.BDBUS6
- new net RS232_RX: R30.1
- new net RS232_TX: R31.1
- new net RTSN: R32.1
- new net VCC1_8FT: C39.1, C40.1, U$1.VCORE0, U$1.VCORE1, U$1.VCORE2, U$1.VREGOUT
- net +3.3V: now also C35.1, C36.1, C37.1, C38.1, R28.2, U$1.VCCIO0, U$1.VCCIO1, U$1.VCCIO2, U$1.VCCIO3, U$1.VPHY, U$1.VPLL, U$1.VREGIN
- net GND: now also C35.2, C36.2, C37.2, C38.2, U$1.AGND, U$1.TEST
Other:
- moved on the sheet: C1, C2, C3, C33, C4, C5, R1, R2, R3, R4, R5, R6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

Commit message: Updated USB-C. Added USB-C to schematic, and the ATSAM3S.
Parts:
- removed U1: ATSAM3S2CA-AU, Atmel_By_element14_Batch_1-00:ATSAM3S2CA-AU
- added U$6: DX07S0, USBC:DX07S0
- added U2: ATSAM3S4AA-AU, Atmel_By_element14_Batch_1-00:ATSAM3S4AA-AU
Connections:
- removed net RS232_RX: R30.1
- removed net RS232_TX: R31.1
- new net DM: U$1.DM, U$6.DN1_A, U$6.DN2_B
- new net DP: U$1.DP, U$6.DP1_A, U$6.DP2_B
- new net URXD0: R30.1, U2.PA9/PGMM1
- new net UTXD0: R31.1, U2.PA10/PGMM2
- net GND: now also U$6.GND2_A, U$6.GND2_B, U$6.GND_A, U$6.GND_B, U2.GND, U2.GND_2; no longer U1.GND, U1.GND_2, U1.GND_3, U1.GND_4, U1.GND_5
- net VBUS_5V: now also U$6.SBU2_B, U$6.VBUS2_A, U$6.VBUS2_B, U$6.VBUS_A

Commit message: Added LEDs to the device table.
Connections:
- new net N$31: U2.ERASE/PB12
Changed lines of the file:
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@@
+</segment>
+</net>
+<net name="N$31" class="0">
+<segment>
+<pinref part="U2" gate="A" pin="ERASE/PB12"/>
+<wire x1="393.7" y1="27.94" x2="411.48" y2="27.94" width="0.1524" layer="91"/>
 </segment>
 </net>

Commit message: Changed LEDs in the device table.
Parts:
- added R37: 1K, resistor:R-US_M1206
Connections:
- removed net N$31: U2.ERASE/PB12
- net DTRN: now also U2.ERASE/PB12
Changed lines of the file:
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@@
 <?xml version="1.0" encoding="utf-8"?>
 <!DOCTYPE eagle SYSTEM "eagle.dtd">
-<eagle version="7.4.0">
+<eagle version="7.3.0">
 <drawing>
 <settings>
@@
 <setting verticaltext="up"/>
 </settings>
-<grid distance="0.1" unitdist="inch" unit="inch" style="lines" multiple="1" display="no" altdistance="0.01" altunitdist="inch" altunit="inch"/>
+<grid distance="0.1" unitdist="inch" unit="inch" style="lines" multiple="1" display="yes" altdistance="0.01" altunitdist="inch" altunit="inch"/>
 <layers>
 <layer number="1" name="Top" color="4" fill="1" visible="no" active="no"/>
@@
 <part name="SUPPLY14" library="supply2" deviceset="GND" device=""/>
 <part name="SUPPLY20" library="supply2" deviceset="GND" device=""/>
+<part name="R37" library="resistor" deviceset="R-US_" device="M1206" value="1K"/>
 </parts>
 <sheets>
@@
 <instance part="SUPPLY14" gate="GND" x="-55.88" y="17.78"/>
 <instance part="SUPPLY20" gate="GND" x="-106.68" y="17.78"/>
+<instance part="R37" gate="G$1" x="287.02" y="208.28" smashed="yes">
+<attribute name="NAME" x="284.48" y="213.868" size="1.778" layer="95" rot="R270"/>
+<attribute name="VALUE" x="287.782" y="213.868" size="1.778" layer="96" rot="R270"/>
+</instance>
 </instances>
 <busses>
@@
 <pinref part="R32" gate="G$1" pin="1"/>
 <wire x1="116.84" y1="104.14" x2="121.92" y2="104.14" width="0.1524" layer="91"/>
-<label x="121.92" y="103.378" size="1.778" layer="95"/>
 </segment>
 </net>
@@
 <pinref part="R33" gate="G$1" pin="1"/>
 <wire x1="116.84" y1="101.6" x2="121.92" y2="101.6" width="0.1524" layer="91"/>
-<label x="121.92" y="100.838" size="1.778" layer="95"/>
 </segment>
 </net>
@@
 <label x="121.92" y="98.298" size="1.778" layer="95"/>
 </segment>
+<segment>
+<pinref part="U2" gate="A" pin="ERASE/PB12"/>
+<wire x1="393.7" y1="27.94" x2="408.94" y2="27.94" width="0.1524" layer="91"/>
+<label x="401.32" y="27.94" size="1.778" layer="95"/>
+</segment>
 </net>
 <net name="DSRN" class="0">
@@
 <pinref part="R35" gate="G$1" pin="1"/>
 <wire x1="116.84" y1="96.52" x2="121.92" y2="96.52" width="0.1524" layer="91"/>
-<label x="121.92" y="95.758" size="1.778" layer="95"/>
 </segment>
 </net>
@@
 <pinref part="R36" gate="G$1" pin="1"/>
 <wire x1="116.84" y1="93.98" x2="121.92" y2="93.98" width="0.1524" layer="91"/>
-<label x="121.92" y="93.218" size="1.778" layer="95"/>
 </segment>
 </net>
@@
 </segment>
 </net>
-<net name="N$31" class="0">
-<segment>
-<pinref part="U2" gate="A" pin="ERASE/PB12"/>
-<wire x1="393.7" y1="27.94" x2="411.48" y2="27.94" width="0.1524" layer="91"/>
-</segment>
-</net>

Commit message: Added blue and red LEDs to device table.
Parts:
- added LED1, LED2: Blue, led:LEDSMT1206
- added LED3, LED4: Green, led:LEDSMT1206
- added LED5, LED6: Amber, led:LEDSMT1206
- added R38, R39, R40, R41, R42: 120, resistor:R-US_M1206
- R37: value 1K -> 120
Connections:
- new net LED1: R37.1, U$2.PIO1_10
- new net LED2: R38.1, U$2.PIO1_11
- new net LED3: R39.1, U$2.PIO1_12
- new net LED4: R40.1, U$2.PIO1_13
- new net LED5: R42.1, U2.PA5/PGMRDY
- new net LED6: R41.1, U2.PA7/XIN32/PGMNVALID
- new net N$31: LED4.A, R40.2
- new net N$32: LED3.A, R39.2
- new net N$33: LED2.A, R38.2
- new net N$34: LED1.A, R37.2
- new net N$36: LED6.A, R42.2
- new net N$37: LED5.A, R41.2
- net GND: now also LED1.C, LED2.C, LED3.C, LED4.C, LED5.C, LED6.C
Other:
- moved on the sheet: R37

Commit message: Removed blue LEDs.
Parts:
- added LED7, LED8: Red, led:LEDSMT1206
- added R43: 25, resistor:R-US_M1206
- added R44: 100, resistor:R-US_M1206
- LED1, LED2: value Blue -> Green
- R37, R38, R39, R40, R41, R42: value 120 -> 100
Connections:
- new net 3.3V: R43.1
- new net N$35: LED8.A, R44.2
- new net N$38: LED7.A, R43.2
- net GND: now also LED7.C, LED8.C
- net VBUS_5V: now also R44.1
Other:
- note added: "FPGA LEDs"
- note added: "MCU LEDs"
Changed lines of the file:
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@@
 <part name="SUPPLY14" library="supply2" deviceset="GND" device=""/>
 <part name="SUPPLY20" library="supply2" deviceset="GND" device=""/>
-<part name="R37" library="resistor" deviceset="R-US_" device="M1206" value="120"/>
-<part name="LED1" library="led" deviceset="LED" device="SMT1206" value="Blue"/>
-<part name="LED2" library="led" deviceset="LED" device="SMT1206" value="Blue"/>
+<part name="R37" library="resistor" deviceset="R-US_" device="M1206" value="100"/>
+<part name="LED1" library="led" deviceset="LED" device="SMT1206" value="Green"/>
+<part name="LED2" library="led" deviceset="LED" device="SMT1206" value="Green"/>
 <part name="LED3" library="led" deviceset="LED" device="SMT1206" value="Green"/>
 <part name="LED4" library="led" deviceset="LED" device="SMT1206" value="Green"/>
-<part name="R38" library="resistor" deviceset="R-US_" device="M1206" value="120"/>
-<part name="R39" library="resistor" deviceset="R-US_" device="M1206" value="120"/>
-<part name="R40" library="resistor" deviceset="R-US_" device="M1206" value="120"/>
+<part name="R38" library="resistor" deviceset="R-US_" device="M1206" value="100"/>
+<part name="R39" library="resistor" deviceset="R-US_" device="M1206" value="100"/>
+<part name="R40" library="resistor" deviceset="R-US_" device="M1206" value="100"/>
 <part name="SUPPLY21" library="supply2" deviceset="GND" device=""/>
 <part name="LED5" library="led" deviceset="LED" device="SMT1206" value="Amber"/>
 <part name="LED6" library="led" deviceset="LED" device="SMT1206" value="Amber"/>
-<part name="R41" library="resistor" deviceset="R-US_" device="M1206" value="120"/>
-<part name="R42" library="resistor" deviceset="R-US_" device="M1206" value="120"/>
+<part name="R41" library="resistor" deviceset="R-US_" device="M1206" value="100"/>
+<part name="R42" library="resistor" deviceset="R-US_" device="M1206" value="100"/>
 <part name="SUPPLY22" library="supply2" deviceset="GND" device=""/>
+<part name="LED7" library="led" deviceset="LED" device="SMT1206" value="Red"/>
+<part name="LED8" library="led" deviceset="LED" device="SMT1206" value="Red"/>
+<part name="R43" library="resistor" deviceset="R-US_" device="M1206" value="25"/>
+<part name="R44" library="resistor" deviceset="R-US_" device="M1206" value="100"/>
+<part name="SUPPLY23" library="supply2" deviceset="GND" device=""/>
 </parts>
 <sheets>
@@
 cap and power pin stuff</text>
 <text x="149.86" y="274.32" size="1.778" layer="91">iCE VCCIOX bypass caps</text>
+<text x="365.76" y="248.92" size="1.778" layer="91">FPGA LEDs</text>
+<text x="368.3" y="195.58" size="1.778" layer="91">MCU LEDs</text>
 </plain>
 <instances>
@@
 <instance part="LED1" gate="G$1" x="381" y="215.9" smashed="yes" rot="R90">
 <attribute name="NAME" x="380.492" y="219.456" size="1.778" layer="95" rot="R180"/>
-<attribute name="VALUE" x="385.572" y="219.075" size="1.778" layer="96" rot="R180"/>
+<attribute name="VALUE" x="388.112" y="219.075" size="1.778" layer="96" rot="R180"/>
 </instance>
 <instance part="LED2" gate="G$1" x="381" y="223.52" smashed="yes" rot="R90">
 <attribute name="NAME" x="380.492" y="227.076" size="1.778" layer="95" rot="R180"/>
-<attribute name="VALUE" x="385.572" y="226.695" size="1.778" layer="96" rot="R180"/>
+<attribute name="VALUE" x="388.112" y="226.695" size="1.778" layer="96" rot="R180"/>
 </instance>
 <instance part="LED3" gate="G$1" x="381" y="231.14" smashed="yes" rot="R90">
@@
 </instance>
 <instance part="SUPPLY22" gate="GND" x="391.16" y="167.64"/>
+<instance part="LED7" gate="G$1" x="-134.62" y="71.12" smashed="yes" rot="R90">
+<attribute name="NAME" x="-135.128" y="74.676" size="1.778" layer="95" rot="R180"/>
+<attribute name="VALUE" x="-127.508" y="74.295" size="1.778" layer="96" rot="R180"/>
+</instance>
+<instance part="LED8" gate="G$1" x="-134.62" y="81.28" smashed="yes" rot="R90">
+<attribute name="NAME" x="-135.128" y="84.836" size="1.778" layer="95" rot="R180"/>
+<attribute name="VALUE" x="-127.508" y="84.455" size="1.778" layer="96" rot="R180"/>
+</instance>
+<instance part="R43" gate="G$1" x="-147.32" y="71.12" smashed="yes">
+<attribute name="NAME" x="-152.4" y="74.168" size="1.778" layer="95"/>
+<attribute name="VALUE" x="-146.558" y="74.168" size="1.778" layer="96"/>
+</instance>
+<instance part="R44" gate="G$1" x="-147.32" y="81.28" smashed="yes">
+<attribute name="NAME" x="-152.4" y="84.328" size="1.778" layer="95"/>
+<attribute name="VALUE" x="-146.558" y="84.328" size="1.778" layer="96"/>
+</instance>
+<instance part="SUPPLY23" gate="GND" x="-124.46" y="63.5"/>
 </instances>
 <busses>
@@
 <pinref part="SUPPLY22" gate="GND" pin="GND"/>
 </segment>
+<segment>
+<pinref part="LED8" gate="G$1" pin="C"/>
+<wire x1="-129.54" y1="81.28" x2="-124.46" y2="81.28" width="0.1524" layer="91"/>
+<wire x1="-124.46" y1="81.28" x2="-124.46" y2="71.12" width="0.1524" layer="91"/>
+<pinref part="LED7" gate="G$1" pin="C"/>
+<wire x1="-129.54" y1="71.12" x2="-124.46" y2="71.12" width="0.1524" layer="91"/>
+<junction x="-124.46" y="71.12"/>
+<pinref part="SUPPLY23" gate="GND" pin="GND"/>
+<wire x1="-124.46" y1="66.04" x2="-124.46" y2="71.12" width="0.1524" layer="91"/>
+</segment>
 </net>
 <net name="N$2" class="0">
@@
 <junction x="-88.9" y="60.96"/>
 <label x="-93.98" y="66.04" size="1.778" layer="95"/>
+</segment>
+<segment>
+<pinref part="R44" gate="G$1" pin="1"/>
+<wire x1="-152.4" y1="81.28" x2="-165.1" y2="81.28" width="0.1524" layer="91"/>
+<label x="-165.1" y="81.28" size="1.778" layer="95"/>
 </segment>
 </net>
@@
 </segment>
 </net>
+<net name="N$35" class="0">
+<segment>
+<pinref part="LED8" gate="G$1" pin="A"/>
+<pinref part="R44" gate="G$1" pin="2"/>
+<wire x1="-137.16" y1="81.28" x2="-142.24" y2="81.28" width="0.1524" layer="91"/>
+</segment>
+</net>
+<net name="N$38" class="0">
+<segment>
+<pinref part="R43" gate="G$1" pin="2"/>
+<pinref part="LED7" gate="G$1" pin="A"/>
+<wire x1="-142.24" y1="71.12" x2="-137.16" y2="71.12" width="0.1524" layer="91"/>
+</segment>
+</net>
+<net name="3.3V" class="0">
+<segment>
+<pinref part="R43" gate="G$1" pin="1"/>
+<wire x1="-152.4" y1="71.12" x2="-165.1" y2="71.12" width="0.1524" layer="91"/>
+<label x="-160.02" y="71.12" size="1.778" layer="95"/>
+</segment>
+</net>

Commit message: Added crystal to schematic.
Parts:
- added C41: 0.1uF, resistor:C-USC0805
- added R45: 100, resistor:R-US_M1206
- added U$7: SG-636PCE, crystal:SG-636PCE
Connections:
- new net 12MHZ: U$7.FO
- new net N$39: R45.1, U$7.OE
- new net N$40: U2.PA3
- new net N$41: U2.PA4/PGMNCMD
- net 3.3V: now also C41.1, R45.2, U$7.VCC, U2.VDDIN, U2.VDDIO, U2.VDDIO_2, U2.VDDIO_3
- net GND: now also C41.2, U$7.GND
Other:
- note added: "12 MHz clock"
Changed lines of the file:
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@@
 <part name="R44" library="resistor" deviceset="R-US_" device="M1206" value="100"/>
 <part name="SUPPLY23" library="supply2" deviceset="GND" device=""/>
+<part name="U$7" library="crystal" deviceset="SG-636PCE" device=""/>
+<part name="SUPPLY24" library="supply2" deviceset="GND" device=""/>
+<part name="C41" library="resistor" deviceset="C-US" device="C0805" value="0.1uF"/>
+<part name="R45" library="resistor" deviceset="R-US_" device="M1206" value="100"/>
 </parts>
 <sheets>
@@
 <text x="365.76" y="248.92" size="1.778" layer="91">FPGA LEDs</text>
 <text x="368.3" y="195.58" size="1.778" layer="91">MCU LEDs</text>
+<text x="27.94" y="256.54" size="1.778" layer="91">12 MHz clock</text>
 </plain>
 <instances>
@@
 </instance>
 <instance part="SUPPLY23" gate="GND" x="-124.46" y="63.5"/>
+<instance part="U$7" gate="G$1" x="35.56" y="243.84"/>
+<instance part="SUPPLY24" gate="GND" x="15.24" y="231.14"/>
+<instance part="C41" gate="G$1" x="15.24" y="243.84"/>
+<instance part="R45" gate="G$1" x="50.8" y="256.54" smashed="yes" rot="R90">
+<attribute name="NAME" x="55.626" y="260.35" size="1.778" layer="95" rot="R180"/>
+<attribute name="VALUE" x="56.642" y="257.81" size="1.778" layer="96" rot="R180"/>
+</instance>
 </instances>
 <busses>
@@
 <wire x1="-124.46" y1="66.04" x2="-124.46" y2="71.12" width="0.1524" layer="91"/>
 </segment>
+<segment>
+<pinref part="U$7" gate="G$1" pin="GND"/>
+<wire x1="22.86" y1="238.76" x2="15.24" y2="238.76" width="0.1524" layer="91"/>
+<wire x1="15.24" y1="238.76" x2="15.24" y2="233.68" width="0.1524" layer="91"/>
+<pinref part="SUPPLY24" gate="GND" pin="GND"/>
+<pinref part="C41" gate="G$1" pin="2"/>
+<junction x="15.24" y="238.76"/>
+</segment>
 </net>
 <net name="N$2" class="0">
@@
 <label x="-160.02" y="71.12" size="1.778" layer="95"/>
 </segment>
-</net>
+<segment>
+<pinref part="U$7" gate="G$1" pin="VCC"/>
+<wire x1="22.86" y1="248.92" x2="15.24" y2="248.92" width="0.1524" layer="91"/>
+<wire x1="15.24" y1="248.92" x2="15.24" y2="251.46" width="0.1524" layer="91"/>
+<label x="12.7" y="251.46" size="1.778" layer="95"/>
+<pinref part="C41" gate="G$1" pin="1"/>
+<wire x1="15.24" y1="246.38" x2="15.24" y2="248.92" width="0.1524" layer="91"/>
+<junction x="15.24" y="248.92"/>
+</segment>
+<segment>
+<pinref part="R45" gate="G$1" pin="2"/>
+<wire x1="50.8" y1="261.62" x2="50.8" y2="266.7" width="0.1524" layer="91"/>
+<label x="48.26" y="266.7" size="1.778" layer="95"/>
+</segment>
+<segment>
+<pinref part="U2" gate="A" pin="VDDIO"/>
+<wire x1="307.34" y1="78.74" x2="302.26" y2="78.74" width="0.1524" layer="91"/>
+<pinref part="U2" gate="A" pin="VDDIO_3"/>
+<wire x1="302.26" y1="78.74" x2="302.26" y2="81.28" width="0.1524" layer="91"/>
+<wire x1="302.26" y1="81.28" x2="307.34" y2="81.28" width="0.1524" layer="91"/>
+<pinref part="U2" gate="A" pin="VDDIO_2"/>
+<wire x1="302.26" y1="81.28" x2="302.26" y2="83.82" width="0.1524" layer="91"/>
+<wire x1="302.26" y1="83.82" x2="307.34" y2="83.82" width="0.1524" layer="91"/>
+<junction x="302.26" y="81.28"/>
+<pinref part="U2" gate="A" pin="VDDIN"/>
+<wire x1="302.26" y1="83.82" x2="302.26" y2="86.36" width="0.1524" layer="91"/>
+<wire x1="302.26" y1="86.36" x2="307.34" y2="86.36" width="0.1524" layer="91"/>
+<junction x="302.26" y="83.82"/>
+<wire x1="302.26" y1="83.82" x2="289.56" y2="83.82" width="0.1524" layer="91"/>
+<wire x1="289.56" y1="83.82" x2="289.56" y2="88.9" width="0.1524" layer="91"/>
+<label x="287.02" y="88.9" size="1.778" layer="95"/>
+</segment>
+</net>
+<net name="N$39" class="0">
+<segment>
+<pinref part="U$7" gate="G$1" pin="OE"/>
+<wire x1="48.26" y1="248.92" x2="50.8" y2="248.92" width="0.1524" layer="91"/>
+<wire x1="50.8" y1="248.92" x2="50.8" y2="251.46" width="0.1524" layer="91"/>
+<pinref part="R45" gate="G$1" pin="1"/>
+</segment>
+</net>
+<net name="12MHZ" class="0">
+<segment>
+<pinref part="U$7" gate="G$1" pin="FO"/>
+<wire x1="48.26" y1="243.84" x2="58.42" y2="243.84" width="0.1524" layer="91"/>
+<label x="55.88" y="243.84" size="1.778" layer="95"/>
+</segment>
+</net>
+<net name="N$40" class="0">
+<segment>
+<pinref part="U2" gate="A" pin="PA3"/>
+<wire x1="393.7" y1="78.74" x2="408.94" y2="78.74" width="0.1524" layer="91"/>
+</segment>
+</net>
+<net name="N$41" class="0">
+<segment>
+<pinref part="U2" gate="A" pin="PA4/PGMNCMD"/>
+<wire x1="393.7" y1="76.2" x2="408.94" y2="76.2" width="0.1524" layer="91"/>
+</segment>
+</net>

Commit message: Added a comment.
Other:
- note added: "Flash for FPGA"
Changed lines of the file:
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@@
 <text x="368.3" y="195.58" size="1.778" layer="91">MCU LEDs</text>
 <text x="27.94" y="256.54" size="1.778" layer="91">12 MHz clock</text>
+<text x="73.66" y="7.62" size="1.778" layer="91">Flash for FPGA</text>
 </plain>
 <instances>
