File: schematic/schematic.sch (EAGLE design)
At the start: 103 parts, among them U2 ATSAM3S4AA-AU

Commit message: Changed package type for all resistors and caps.
Parts:
- added C42, C45, C46: 10uF, resistor:C-USC0603
- added C43: 2.2uF, resistor:C-USC0603
- added C44, C47, C48: 0.1uF, resistor:C-USC0603
- C1, C10, C11, C12, C13, C14, C15, C16, C17, C18, C19, C2, C20, C21, C22, C23, C24, C25, C26, C27, C28, C29, C3, C30, C31, C32, C33, C34, C35, C36, C37, C38, C39, C4, C40, C41, C5, C6, C7, C8, C9: device resistor:C-USC0805 -> resistor:C-USC0603
- R1, R10, R11, R12, R13, R14, R15, R16, R17, R18, R19, R2, R20, R21, R22, R23, R24, R25, R26, R27, R28, R29, R3, R30, R31, R32, R33, R34, R35, R36, R37, R38, R39, R4, R40, R41, R42, R43, R44, R45, R5, R6, R7, R8, R9: device resistor:R-US_M1206 -> resistor:R-US_R0603
Connections:
- removed net N$41: U2.PA4/PGMNCMD
- net 3.3V: now also C42.1, C43.1, C44.1, C45.1, C46.1, C47.1, C48.1
- net GND: now also C42.2, C43.2, C44.2, C45.2, C46.2, C47.2, C48.2
- net N$40: now also U2.VDDCORE, U2.VDDCORE_2, U2.VDDOUT; no longer U2.PA3
Other:
- note added: "For Vin"
- note added: "For Vout"

Commit message: Added bypass caps for MCU.
Parts:
- added C49, C51: 10uF, resistor:C-USC0603
- added C50, C52: 0.1uF, resistor:C-USC0603
Connections:
- net 3.3V: now also C49.1, C50.1, C51.1, C52.1
- net GND: now also C49.2, C50.2, C51.2, C52.2
Other:
- moved on the sheet: C45, C46, C47, C48

Commit message: Updated schematice comments.
Other:
- note added: "For VDDin"
- note added: "For VDDout"
- note removed: "For Vin"
- note removed: "For Vout"
Changed lines of the file:
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@@
 <text x="27.94" y="256.54" size="1.778" layer="91">12 MHz clock</text>
 <text x="73.66" y="7.62" size="1.778" layer="91">Flash for FPGA</text>
-<text x="314.96" y="116.84" size="1.778" layer="91" rot="R90">For Vin</text>
-<text x="335.28" y="124.46" size="1.778" layer="91" rot="R270">For Vout</text>
+<text x="314.96" y="116.84" size="1.778" layer="91" rot="R90">For VDDin</text>
+<text x="340.36" y="127" size="1.778" layer="91">For VDDout</text>
 </plain>
 <instances>

Commit message: Added crystal for the MCU.
Parts:
- added C53, C54: 56pF, resistor:C-USC0603
- added Q1: (no value), crystal:CRYSTALHC49UP
Connections:
- new net XIN: C53.1, Q1.2, U2.XIN/PB9/PGMCK
- new net XOUT: C54.1, Q1.1, U2.XOUT/PB8
- net GND: now also C53.2, C54.2
Changed lines of the file:
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@@
 <part name="C51" library="resistor" deviceset="C-US" device="C0603" value="10uF"/>
 <part name="C52" library="resistor" deviceset="C-US" device="C0603" value="0.1uF"/>
+<part name="Q1" library="crystal" deviceset="CRYSTAL" device="HC49UP"/>
+<part name="C53" library="resistor" deviceset="C-US" device="C0603" value="56pF"/>
+<part name="C54" library="resistor" deviceset="C-US" device="C0603" value="56pF"/>
+<part name="SUPPLY27" library="supply2" deviceset="GND" device=""/>
+<part name="SUPPLY28" library="supply2" deviceset="GND" device=""/>
 </parts>
 <sheets>
@@
 <instance part="C51" gate="G$1" x="406.4" y="137.16"/>
 <instance part="C52" gate="G$1" x="482.6" y="137.16"/>
+<instance part="Q1" gate="G$1" x="467.36" y="83.82" rot="R180"/>
+<instance part="C53" gate="G$1" x="457.2" y="73.66"/>
+<instance part="C54" gate="G$1" x="477.52" y="73.66"/>
+<instance part="SUPPLY27" gate="GND" x="457.2" y="60.96"/>
+<instance part="SUPPLY28" gate="GND" x="477.52" y="60.96"/>
 </instances>
 <busses>
@@
 <junction x="472.44" y="129.54"/>
 </segment>
+<segment>
+<pinref part="SUPPLY27" gate="GND" pin="GND"/>
+<pinref part="C53" gate="G$1" pin="2"/>
+<wire x1="457.2" y1="63.5" x2="457.2" y2="68.58" width="0.1524" layer="91"/>
+</segment>
+<segment>
+<pinref part="SUPPLY28" gate="GND" pin="GND"/>
+<pinref part="C54" gate="G$1" pin="2"/>
+<wire x1="477.52" y1="63.5" x2="477.52" y2="68.58" width="0.1524" layer="91"/>
+</segment>
 </net>
 <net name="N$2" class="0">
@@
 </segment>
 </net>
+<net name="XIN" class="0">
+<segment>
+<pinref part="Q1" gate="G$1" pin="2"/>
+<wire x1="457.2" y1="83.82" x2="464.82" y2="83.82" width="0.1524" layer="91"/>
+<pinref part="C53" gate="G$1" pin="1"/>
+<wire x1="457.2" y1="76.2" x2="457.2" y2="83.82" width="0.1524" layer="91"/>
+<wire x1="457.2" y1="83.82" x2="457.2" y2="91.44" width="0.1524" layer="91"/>
+<junction x="457.2" y="83.82"/>
+<label x="454.66" y="91.44" size="1.778" layer="95"/>
+</segment>
+<segment>
+<pinref part="U2" gate="A" pin="XIN/PB9/PGMCK"/>
+<wire x1="307.34" y1="60.96" x2="297.18" y2="60.96" width="0.1524" layer="91"/>
+<label x="297.18" y="60.96" size="1.778" layer="95"/>
+</segment>
+</net>
+<net name="XOUT" class="0">
+<segment>
+<pinref part="Q1" gate="G$1" pin="1"/>
+<wire x1="477.52" y1="83.82" x2="469.9" y2="83.82" width="0.1524" layer="91"/>
+<pinref part="C54" gate="G$1" pin="1"/>
+<wire x1="477.52" y1="76.2" x2="477.52" y2="83.82" width="0.1524" layer="91"/>
+<wire x1="477.52" y1="83.82" x2="477.52" y2="91.44" width="0.1524" layer="91"/>
+<junction x="477.52" y="83.82"/>
+<label x="474.98" y="91.44" size="1.778" layer="95"/>
+</segment>
+<segment>
+<pinref part="U2" gate="A" pin="XOUT/PB8"/>
+<wire x1="307.34" y1="35.56" x2="297.18" y2="35.56" width="0.1524" layer="91"/>
+<label x="297.18" y="35.56" size="1.778" layer="95"/>
+</segment>
+</net>

Commit message: Added some connections between the FPGA and the MCU.
Parts:
- added R46, R47: 1k, resistor:R-US_R0603
Connections:
- new net IO1: U2.DDM/PB10
- new net IO2: U2.DDP/PB11
- new net M_MISO: U$2.PIO2_13, U2.PA12/PGMD0
- new net M_MOSI: U$2.PIO2_12, U2.PA13/PGMD1
- new net M_SPCK: U$2.GBIN5/PIO2_01, U2.PA14/PGMD2
- new net SPI_NPCS0: U$2.PIO2_11, U2.PA11/PGMM3
- new net SPI_NPCS1: U$2.PIO2_10
- new net SPI_NPCS2: U$2.PIO2_09
- new net TWCK0: R47.1, U2.PA4/PGMNCMD
- new net TWD0: R46.1, U2.PA3
- new net URXD1: U$2.PIO3_08/DP03A, U2.PB3/AD7
- new net UTXD1: U$2.PIO3_09/DP03B, U2.PB2/AD6
- net 3.3V: now also R46.2, R47.2
Changed lines of the file:
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@@
 <setting verticaltext="up"/>
 </settings>
-<grid distance="0.1" unitdist="inch" unit="inch" style="lines" multiple="1" display="no" altdistance="0.01" altunitdist="inch" altunit="inch"/>
+<grid distance="0.1" unitdist="inch" unit="inch" style="lines" multiple="1" display="yes" altdistance="0.01" altunitdist="inch" altunit="inch"/>
 <layers>
 <layer number="1" name="Top" color="4" fill="1" visible="no" active="no"/>
@@
 <part name="SUPPLY27" library="supply2" deviceset="GND" device=""/>
 <part name="SUPPLY28" library="supply2" deviceset="GND" device=""/>
+<part name="R46" library="resistor" deviceset="R-US_" device="R0603" value="1k"/>
+<part name="R47" library="resistor" deviceset="R-US_" device="R0603" value="1k"/>
 </parts>
 <sheets>
@@
 <instance part="SUPPLY27" gate="GND" x="457.2" y="60.96"/>
 <instance part="SUPPLY28" gate="GND" x="477.52" y="60.96"/>
+<instance part="R46" gate="G$1" x="419.1" y="86.36" smashed="yes" rot="R90">
+<attribute name="NAME" x="416.56" y="85.852" size="1.778" layer="95" rot="R180"/>
+<attribute name="VALUE" x="415.798" y="88.392" size="1.778" layer="96" rot="R180"/>
+</instance>
+<instance part="R47" gate="G$1" x="426.72" y="86.36" smashed="yes" rot="R90">
+<attribute name="NAME" x="434.34" y="85.852" size="1.778" layer="95" rot="R180"/>
+<attribute name="VALUE" x="433.578" y="88.392" size="1.778" layer="96" rot="R180"/>
+</instance>
 </instances>
 <busses>
@@
 <junction x="472.44" y="142.24"/>
 </segment>
+<segment>
+<pinref part="R46" gate="G$1" pin="2"/>
+<wire x1="419.1" y1="91.44" x2="419.1" y2="93.98" width="0.1524" layer="91"/>
+<wire x1="419.1" y1="93.98" x2="426.72" y2="93.98" width="0.1524" layer="91"/>
+<pinref part="R47" gate="G$1" pin="2"/>
+<wire x1="426.72" y1="93.98" x2="426.72" y2="91.44" width="0.1524" layer="91"/>
+<label x="421.64" y="93.98" size="1.778" layer="95"/>
+</segment>
 </net>
 <net name="N$39" class="0">
@@
 </segment>
 </net>
+<net name="M_SPCK" class="0">
+<segment>
+<pinref part="U$2" gate="G$1" pin="GBIN5/PIO2_01"/>
+<wire x1="233.68" y1="88.9" x2="246.38" y2="88.9" width="0.1524" layer="91"/>
+<label x="241.3" y="88.9" size="1.778" layer="95"/>
+</segment>
+<segment>
+<pinref part="U2" gate="A" pin="PA14/PGMD2"/>
+<wire x1="393.7" y1="50.8" x2="414.02" y2="50.8" width="0.1524" layer="91"/>
+<label x="403.86" y="50.8" size="1.778" layer="95"/>
+</segment>
+</net>
+<net name="M_MOSI" class="0">
+<segment>
+<pinref part="U$2" gate="G$1" pin="PIO2_12"/>
+<wire x1="233.68" y1="60.96" x2="256.54" y2="60.96" width="0.1524" layer="91"/>
+<label x="241.3" y="60.96" size="1.778" layer="95"/>
+</segment>
+<segment>
+<pinref part="U2" gate="A" pin="PA13/PGMD1"/>
+<wire x1="393.7" y1="53.34" x2="414.02" y2="53.34" width="0.1524" layer="91"/>
+<label x="403.86" y="53.34" size="1.778" layer="95"/>
+</segment>
+</net>
+<net name="SPI_NPCS0" class="0">
+<segment>
+<pinref part="U$2" gate="G$1" pin="PIO2_11"/>
+<wire x1="233.68" y1="63.5" x2="256.54" y2="63.5" width="0.1524" layer="91"/>
+<label x="241.3" y="63.5" size="1.778" layer="95"/>
+</segment>
+<segment>
+<pinref part="U2" gate="A" pin="PA11/PGMM3"/>
+<wire x1="393.7" y1="58.42" x2="414.02" y2="58.42" width="0.1524" layer="91"/>
+<label x="401.32" y="58.42" size="1.778" layer="95"/>
+</segment>
+</net>
+<net name="SPI_NPCS1" class="0">
+<segment>
+<pinref part="U$2" gate="G$1" pin="PIO2_10"/>
+<wire x1="233.68" y1="66.04" x2="256.54" y2="66.04" width="0.1524" layer="91"/>
+<label x="241.3" y="66.04" size="1.778" layer="95"/>
+</segment>
+</net>
+<net name="SPI_NPCS2" class="0">
+<segment>
+<pinref part="U$2" gate="G$1" pin="PIO2_09"/>
+<wire x1="233.68" y1="68.58" x2="256.54" y2="68.58" width="0.1524" layer="91"/>
+<label x="241.3" y="68.58" size="1.778" layer="95"/>
+</segment>
+</net>
+<net name="M_MISO" class="0">
+<segment>
+<pinref part="U$2" gate="G$1" pin="PIO2_13"/>
+<wire x1="233.68" y1="58.42" x2="256.54" y2="58.42" width="0.1524" layer="91"/>
+<label x="241.3" y="58.42" size="1.778" layer="95"/>
+</segment>
+<segment>
+<pinref part="U2" gate="A" pin="PA12/PGMD0"/>
+<wire x1="393.7" y1="55.88" x2="414.02" y2="55.88" width="0.1524" layer="91"/>
+<label x="403.86" y="55.88" size="1.778" layer="95"/>
+</segment>
+</net>
+<net name="URXD1" class="0">
+<segment>
+<pinref part="U$2" gate="G$1" pin="PIO3_08/DP03A"/>
+<wire x1="233.68" y1="15.24" x2="246.38" y2="15.24" width="0.1524" layer="91"/>
+<label x="238.76" y="15.24" size="1.778" layer="95"/>
+</segment>
+<segment>
+<pinref part="U2" gate="A" pin="PB3/AD7"/>
+<wire x1="307.34" y1="48.26" x2="297.18" y2="48.26" width="0.1524" layer="91"/>
+<label x="297.18" y="48.26" size="1.778" layer="95"/>
+</segment>
+</net>
+<net name="UTXD1" class="0">
+<segment>
+<pinref part="U$2" gate="G$1" pin="PIO3_09/DP03B"/>
+<wire x1="233.68" y1="12.7" x2="246.38" y2="12.7" width="0.1524" layer="91"/>
+<label x="238.76" y="12.7" size="1.778" layer="95"/>
+</segment>
+<segment>
+<pinref part="U2" gate="A" pin="PB2/AD6"/>
+<wire x1="307.34" y1="50.8" x2="297.18" y2="50.8" width="0.1524" layer="91"/>
+<label x="297.18" y="50.8" size="1.778" layer="95"/>
+</segment>
+</net>
+<net name="IO1" class="0">
+<segment>
+<pinref part="U2" gate="A" pin="DDM/PB10"/>
+<wire x1="307.34" y1="33.02" x2="297.18" y2="33.02" width="0.1524" layer="91"/>
+<label x="297.18" y="33.02" size="1.778" layer="95"/>
+</segment>
+</net>
+<net name="IO2" class="0">
+<segment>
+<pinref part="U2" gate="A" pin="DDP/PB11"/>
+<wire x1="393.7" y1="30.48" x2="408.94" y2="30.48" width="0.1524" layer="91"/>
+<label x="403.86" y="30.48" size="1.778" layer="95"/>
+</segment>
+</net>
+<net name="TWD0" class="0">
+<segment>
+<pinref part="U2" gate="A" pin="PA3"/>
+<wire x1="393.7" y1="78.74" x2="419.1" y2="78.74" width="0.1524" layer="91"/>
+<label x="429.26" y="78.74" size="1.778" layer="95"/>
+<pinref part="R46" gate="G$1" pin="1"/>
+<wire x1="419.1" y1="78.74" x2="419.1" y2="81.28" width="0.1524" layer="91"/>
+<wire x1="419.1" y1="78.74" x2="436.88" y2="78.74" width="0.1524" layer="91"/>
+<junction x="419.1" y="78.74"/>
+</segment>
+</net>
+<net name="TWCK0" class="0">
+<segment>
+<pinref part="U2" gate="A" pin="PA4/PGMNCMD"/>
+<label x="429.26" y="76.2" size="1.778" layer="95"/>
+<pinref part="R47" gate="G$1" pin="1"/>
+<wire x1="426.72" y1="81.28" x2="426.72" y2="76.2" width="0.1524" layer="91"/>
+<wire x1="426.72" y1="76.2" x2="393.7" y2="76.2" width="0.1524" layer="91"/>
+<wire x1="426.72" y1="76.2" x2="436.88" y2="76.2" width="0.1524" layer="91"/>
+<junction x="426.72" y="76.2"/>
+</segment>
+</net>

Commit message: Added GPIO between the MCU and the FPGA.
Connections:
- new net AD0: U2.PA17/PGMD5/AD0
- new net AD1: U2.PA18/PGMD6/AD1
- new net AD2: U2.PA19/PGMD7/AD2
- new net AD3: U2.PA20/AD3
- new net AD4: U2.PB0/AD4
- new net AD5: U2.PB1/AD5
- new net GPIO0: U$2.PIO3_11/DP04B, U2.PA0/PGMEN0
- new net GPIO1: U$2.PIO3_12/DP07A, U2.PA1/PGMEN1
- new net GPIO2: U$2.GBIN7/PIO3_01/DP07B, U2.PA2/PGMEN2
- new net GPIO3: U$2.GBIN6/PIO3_00/DP08A, U2.PA6/PGMNOE
- new net GPIO4: U$2.PIO3_13/DP08B, U2.PA8/XOUT32/PGMM0
- new net GPIO5: U$2.PIO3_14/DP09A, U2.PA15/PGMD3
- new net GPIO6: U$2.PIO3_15/DP09B, U2.PA16/PGMD4
Other:
- note added: "AD still need connected to external pins"
Changed lines of the file:
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@@
 <?xml version="1.0" encoding="utf-8"?>
 <!DOCTYPE eagle SYSTEM "eagle.dtd">
-<eagle version="7.4.0">
+<eagle version="7.3.0">
 <drawing>
 <settings>
@@
 <text x="314.96" y="116.84" size="1.778" layer="91" rot="R90">For VDDin</text>
 <text x="340.36" y="127" size="1.778" layer="91">For VDDout</text>
+<text x="429.26" y="40.64" size="1.778" layer="91">AD still need connected to external pins</text>
 </plain>
 <instances>
@@
 </segment>
 </net>
+<net name="AD4" class="0">
+<segment>
+<pinref part="U2" gate="A" pin="PB0/AD4"/>
+<wire x1="307.34" y1="55.88" x2="297.18" y2="55.88" width="0.1524" layer="91"/>
+<label x="297.18" y="55.88" size="1.778" layer="95"/>
+</segment>
+</net>
+<net name="AD5" class="0">
+<segment>
+<pinref part="U2" gate="A" pin="PB1/AD5"/>
+<wire x1="307.34" y1="53.34" x2="297.18" y2="53.34" width="0.1524" layer="91"/>
+<label x="297.18" y="53.34" size="1.778" layer="95"/>
+</segment>
+</net>
+<net name="AD0" class="0">
+<segment>
+<pinref part="U2" gate="A" pin="PA17/PGMD5/AD0"/>
+<wire x1="393.7" y1="43.18" x2="414.02" y2="43.18" width="0.1524" layer="91"/>
+<label x="408.94" y="43.18" size="1.778" layer="95"/>
+</segment>
+</net>
+<net name="AD1" class="0">
+<segment>
+<pinref part="U2" gate="A" pin="PA18/PGMD6/AD1"/>
+<wire x1="393.7" y1="40.64" x2="414.02" y2="40.64" width="0.1524" layer="91"/>
+<label x="408.94" y="40.64" size="1.778" layer="95"/>
+</segment>
+</net>
+<net name="AD2" class="0">
+<segment>
+<pinref part="U2" gate="A" pin="PA19/PGMD7/AD2"/>
+<wire x1="393.7" y1="38.1" x2="414.02" y2="38.1" width="0.1524" layer="91"/>
+<label x="408.94" y="38.1" size="1.778" layer="95"/>
+</segment>
+</net>
+<net name="AD3" class="0">
+<segment>
+<pinref part="U2" gate="A" pin="PA20/AD3"/>
+<wire x1="393.7" y1="35.56" x2="414.02" y2="35.56" width="0.1524" layer="91"/>
+<label x="408.94" y="35.56" size="1.778" layer="95"/>
+</segment>
+</net>
+<net name="GPIO0" class="0">
+<segment>
+<pinref part="U2" gate="A" pin="PA0/PGMEN0"/>
+<wire x1="393.7" y1="86.36" x2="406.4" y2="86.36" width="0.1524" layer="91"/>
+<label x="398.78" y="86.36" size="1.778" layer="95"/>
+</segment>
+<segment>
+<pinref part="U$2" gate="G$1" pin="PIO3_11/DP04B"/>
+<wire x1="233.68" y1="7.62" x2="246.38" y2="7.62" width="0.1524" layer="91"/>
+<label x="238.76" y="7.62" size="1.778" layer="95"/>
+</segment>
+</net>
+<net name="GPIO1" class="0">
+<segment>
+<pinref part="U2" gate="A" pin="PA1/PGMEN1"/>
+<wire x1="393.7" y1="83.82" x2="406.4" y2="83.82" width="0.1524" layer="91"/>
+<label x="398.78" y="83.82" size="1.778" layer="95"/>
+</segment>
+<segment>
+<pinref part="U$2" gate="G$1" pin="PIO3_12/DP07A"/>
+<wire x1="233.68" y1="5.08" x2="246.38" y2="5.08" width="0.1524" layer="91"/>
+<label x="238.76" y="5.08" size="1.778" layer="95"/>
+</segment>
+</net>
+<net name="GPIO2" class="0">
+<segment>
+<pinref part="U2" gate="A" pin="PA2/PGMEN2"/>
+<wire x1="393.7" y1="81.28" x2="406.4" y2="81.28" width="0.1524" layer="91"/>
+<label x="398.78" y="81.28" size="1.778" layer="95"/>
+</segment>
+<segment>
+<pinref part="U$2" gate="G$1" pin="GBIN7/PIO3_01/DP07B"/>
+<wire x1="233.68" y1="33.02" x2="246.38" y2="33.02" width="0.1524" layer="91"/>
+<label x="238.76" y="33.02" size="1.778" layer="95"/>
+</segment>
+</net>
+<net name="GPIO3" class="0">
+<segment>
+<pinref part="U2" gate="A" pin="PA6/PGMNOE"/>
+<wire x1="393.7" y1="71.12" x2="408.94" y2="71.12" width="0.1524" layer="91"/>
+<label x="401.32" y="71.12" size="1.778" layer="95"/>
+</segment>
+<segment>
+<pinref part="U$2" gate="G$1" pin="GBIN6/PIO3_00/DP08A"/>
+<wire x1="233.68" y1="35.56" x2="246.38" y2="35.56" width="0.1524" layer="91"/>
+<label x="238.76" y="35.56" size="1.778" layer="95"/>
+</segment>
+</net>
+<net name="GPIO4" class="0">
+<segment>
+<pinref part="U2" gate="A" pin="PA8/XOUT32/PGMM0"/>
+<wire x1="393.7" y1="66.04" x2="408.94" y2="66.04" width="0.1524" layer="91"/>
+<label x="401.32" y="66.04" size="1.778" layer="95"/>
+</segment>
+<segment>
+<pinref part="U$2" gate="G$1" pin="PIO3_13/DP08B"/>
+<wire x1="233.68" y1="2.54" x2="246.38" y2="2.54" width="0.1524" layer="91"/>
+<label x="238.76" y="2.54" size="1.778" layer="95"/>
+</segment>
+</net>
+<net name="GPIO5" class="0">
+<segment>
+<pinref part="U2" gate="A" pin="PA15/PGMD3"/>
+<wire x1="393.7" y1="48.26" x2="414.02" y2="48.26" width="0.1524" layer="91"/>
+<label x="406.4" y="48.26" size="1.778" layer="95"/>
+</segment>
+<segment>
+<pinref part="U$2" gate="G$1" pin="PIO3_14/DP09A"/>
+<wire x1="233.68" y1="0" x2="246.38" y2="0" width="0.1524" layer="91"/>
+<label x="238.76" y="0" size="1.778" layer="95"/>
+</segment>
+</net>
+<net name="GPIO6" class="0">
+<segment>
+<pinref part="U2" gate="A" pin="PA16/PGMD4"/>
+<wire x1="393.7" y1="45.72" x2="414.02" y2="45.72" width="0.1524" layer="91"/>
+<label x="406.4" y="45.72" size="1.778" layer="95"/>
+</segment>
+<segment>
+<pinref part="U$2" gate="G$1" pin="PIO3_15/DP09B"/>
+<wire x1="233.68" y1="-2.54" x2="246.38" y2="-2.54" width="0.1524" layer="91"/>
+<label x="238.76" y="-2.54" size="1.778" layer="95"/>
+</segment>
+</net>

Commit message: Fixed bug with NPCSx connections.
Connections:
- removed net SPI_NPCS1: U$2.PIO2_10
- removed net SPI_NPCS2: U$2.PIO2_09
Changed lines of the file:
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@@
 <segment>
 <pinref part="U2" gate="A" pin="PA9/PGMM1"/>
-<wire x1="393.7" y1="63.5" x2="408.94" y2="63.5" width="0.1524" layer="91"/>
-<label x="401.32" y="63.5" size="1.778" layer="95"/>
+<wire x1="393.7" y1="63.5" x2="411.48" y2="63.5" width="0.1524" layer="91"/>
+<label x="403.86" y="63.5" size="1.778" layer="95"/>
 </segment>
 <segment>
@@
 <segment>
 <pinref part="U2" gate="A" pin="PA10/PGMM2"/>
-<wire x1="393.7" y1="60.96" x2="408.94" y2="60.96" width="0.1524" layer="91"/>
-<label x="401.32" y="60.96" size="1.778" layer="95"/>
+<wire x1="393.7" y1="60.96" x2="411.48" y2="60.96" width="0.1524" layer="91"/>
+<label x="403.86" y="60.96" size="1.778" layer="95"/>
 </segment>
 <segment>
@@
 <segment>
 <pinref part="U2" gate="A" pin="PA5/PGMRDY"/>
-<wire x1="393.7" y1="73.66" x2="408.94" y2="73.66" width="0.1524" layer="91"/>
+<wire x1="393.7" y1="73.66" x2="411.48" y2="73.66" width="0.1524" layer="91"/>
 <label x="403.86" y="73.66" size="1.778" layer="95"/>
 </segment>
@@
 <segment>
 <pinref part="U2" gate="A" pin="PA7/XIN32/PGMNVALID"/>
-<wire x1="393.7" y1="68.58" x2="408.94" y2="68.58" width="0.1524" layer="91"/>
+<wire x1="393.7" y1="68.58" x2="411.48" y2="68.58" width="0.1524" layer="91"/>
 <label x="403.86" y="68.58" size="1.778" layer="95"/>
 </segment>
@@
 </segment>
 </net>
-<net name="SPI_NPCS1" class="0">
-<segment>
-<pinref part="U$2" gate="G$1" pin="PIO2_10"/>
-<wire x1="233.68" y1="66.04" x2="256.54" y2="66.04" width="0.1524" layer="91"/>
-<label x="241.3" y="66.04" size="1.778" layer="95"/>
-</segment>
-</net>
-<net name="SPI_NPCS2" class="0">
-<segment>
-<pinref part="U$2" gate="G$1" pin="PIO2_09"/>
-<wire x1="233.68" y1="68.58" x2="256.54" y2="68.58" width="0.1524" layer="91"/>
-<label x="241.3" y="68.58" size="1.778" layer="95"/>
-</segment>
-</net>
 <net name="M_MISO" class="0">
 <segment>
@@
 <segment>
 <pinref part="U2" gate="A" pin="PA15/PGMD3"/>
-<wire x1="393.7" y1="48.26" x2="414.02" y2="48.26" width="0.1524" layer="91"/>
-<label x="406.4" y="48.26" size="1.778" layer="95"/>
+<wire x1="393.7" y1="48.26" x2="411.48" y2="48.26" width="0.1524" layer="91"/>
+<label x="403.86" y="48.26" size="1.778" layer="95"/>
 </segment>
 <segment>
@@
 <segment>
 <pinref part="U2" gate="A" pin="PA16/PGMD4"/>
-<wire x1="393.7" y1="45.72" x2="414.02" y2="45.72" width="0.1524" layer="91"/>
-<label x="406.4" y="45.72" size="1.778" layer="95"/>
-</segment>
-<segment>
+<wire x1="393.7" y1="45.72" x2="411.48" y2="45.72" width="0.1524" layer="91"/>
+<label x="403.86" y="45.72" size="1.778" layer="95"/>
+</segment>
+<segment>

Commit message: Connected the TWI interface.
Connections:
- removed net IO1: U2.DDM/PB10
- removed net IO2: U2.DDP/PB11
- new net GPIO7: U$2.PIO3_16/DP10A, U2.DDM/PB10
- new net GPIO8: U$2.PIO3_17/DP10B, U2.DDP/PB11
- net 12MHZ: now also U$2.GBIN0/PIO0_00
- net TWCK0: now also U$2.PIO3_04/DP01A
- net TWD0: now also U$2.PIO3_03/DP00B
Changed lines of the file:
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@@
 <setting verticaltext="up"/>
 </settings>
-<grid distance="0.1" unitdist="inch" unit="inch" style="lines" multiple="1" display="yes" altdistance="0.01" altunitdist="inch" altunit="inch"/>
+<grid distance="0.1" unitdist="inch" unit="inch" style="lines" multiple="1" display="no" altdistance="0.01" altunitdist="inch" altunit="inch"/>
 <layers>
 <layer number="1" name="Top" color="4" fill="1" visible="no" active="no"/>
@@
 <label x="55.88" y="243.84" size="1.778" layer="95"/>
 </segment>
+<segment>
+<pinref part="U$2" gate="G$1" pin="GBIN0/PIO0_00"/>
+<wire x1="233.68" y1="223.52" x2="246.38" y2="223.52" width="0.1524" layer="91"/>
+</segment>
 </net>
 <net name="N$40" class="0">
@@
 </segment>
 </net>
-<net name="IO1" class="0">
+<net name="GPIO7" class="0">
 <segment>
 <pinref part="U2" gate="A" pin="DDM/PB10"/>
@@
 <label x="297.18" y="33.02" size="1.778" layer="95"/>
 </segment>
-</net>
-<net name="IO2" class="0">
+<segment>
+<pinref part="U$2" gate="G$1" pin="PIO3_16/DP10A"/>
+<wire x1="233.68" y1="-5.08" x2="246.38" y2="-5.08" width="0.1524" layer="91"/>
+<label x="238.76" y="-5.08" size="1.778" layer="95"/>
+</segment>
+</net>
+<net name="GPIO8" class="0">
 <segment>
 <pinref part="U2" gate="A" pin="DDP/PB11"/>
 <wire x1="393.7" y1="30.48" x2="408.94" y2="30.48" width="0.1524" layer="91"/>
-<label x="403.86" y="30.48" size="1.778" layer="95"/>
+<label x="401.32" y="30.48" size="1.778" layer="95"/>
+</segment>
+<segment>
+<pinref part="U$2" gate="G$1" pin="PIO3_17/DP10B"/>
+<wire x1="233.68" y1="-7.62" x2="246.38" y2="-7.62" width="0.1524" layer="91"/>
+<label x="238.76" y="-7.62" size="1.778" layer="95"/>
 </segment>
 </net>
@@
 <junction x="419.1" y="78.74"/>
 </segment>
+<segment>
+<pinref part="U$2" gate="G$1" pin="PIO3_03/DP00B"/>
+<wire x1="233.68" y1="27.94" x2="246.38" y2="27.94" width="0.1524" layer="91"/>
+<label x="238.76" y="27.94" size="1.778" layer="95"/>
+</segment>
 </net>
 <net name="TWCK0" class="0">
@@
 <junction x="426.72" y="76.2"/>
 </segment>
-</net>
+<segment>
+<pinref part="U$2" gate="G$1" pin="PIO3_04/DP01A"/>
+<wire x1="233.68" y1="25.4" x2="246.38" y2="25.4" width="0.1524" layer="91"/>
+<label x="238.76" y="25.4" size="1.778" layer="95"/>
+</segment>
+</net>
