File: schematic/schematic.sch (EAGLE design)
At the start: 119 parts, among them U2 ATSAM3S4AA-AU

Commit message: Added ADVREF.
Connections:
- new net ADVREF: U2.ADVREF
Other:
- note added: "ADx and ADVREF still need connected to external pins"
- note removed: "AD still need connected to external pins"
Changed lines of the file:
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@@
 <setting verticaltext="up"/>
 </settings>
-<grid distance="0.1" unitdist="inch" unit="inch" style="lines" multiple="1" display="no" altdistance="0.01" altunitdist="inch" altunit="inch"/>
+<grid distance="0.1" unitdist="inch" unit="inch" style="lines" multiple="1" display="yes" altdistance="0.01" altunitdist="inch" altunit="inch"/>
 <layers>
 <layer number="1" name="Top" color="4" fill="1" visible="no" active="no"/>
@@
 <text x="314.96" y="116.84" size="1.778" layer="91" rot="R90">For VDDin</text>
 <text x="340.36" y="127" size="1.778" layer="91">For VDDout</text>
-<text x="429.26" y="40.64" size="1.778" layer="91">AD still need connected to external pins</text>
+<text x="429.26" y="40.64" size="1.778" layer="91">ADx and ADVREF still need connected to external pins</text>
 </plain>
 <instances>
@@
 <pinref part="U$2" gate="G$1" pin="GBIN0/PIO0_00"/>
 <wire x1="233.68" y1="223.52" x2="246.38" y2="223.52" width="0.1524" layer="91"/>
+<label x="238.76" y="223.52" size="1.778" layer="95"/>
 </segment>
 </net>
@@
 </segment>
 </net>
+<net name="ADVREF" class="0">
+<segment>
+<pinref part="U2" gate="A" pin="ADVREF"/>
+<wire x1="307.34" y1="68.58" x2="297.18" y2="68.58" width="0.1524" layer="91"/>
+<label x="297.18" y="68.58" size="1.778" layer="95"/>
+</segment>
+</net>

Commit message: Added Vddpll wire.
Connections:
- net N$40: now also U2.VDDPLL
Changed lines of the file:
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@@
 <wire x1="297.18" y1="91.44" x2="307.34" y2="91.44" width="0.1524" layer="91"/>
 <junction x="297.18" y="88.9"/>
+<pinref part="U2" gate="A" pin="VDDPLL"/>
+<wire x1="297.18" y1="76.2" x2="297.18" y2="73.66" width="0.1524" layer="91"/>
+<wire x1="297.18" y1="73.66" x2="307.34" y2="73.66" width="0.1524" layer="91"/>
+<junction x="297.18" y="76.2"/>
 </segment>
 </net>

Commit message: Added the connectors
Parts:
- added JP1, JP2, JP3, JP4, JP5: (no value), SparkFun-Connectors:M06SILK_FEMALE_PTH
- added R48: 0, resistor:R-US_R0603
Connections:
- new net IOA0: JP1.1, U$2.PIO0_02
- new net IOA1: JP1.2, U$2.PIO0_03
- new net IOA2: JP1.3, U$2.PIO0_04
- new net IOA3: JP1.4, U$2.PIO0_05
- new net IOB0: JP2.1, U$2.PIO0_07
- new net IOB1: JP2.2, U$2.PIO0_08
- new net IOB2: JP2.3, U$2.PIO0_09
- new net IOB3: JP2.4, U$2.PIO0_10
- new net IOC0: JP3.1, U$2.PIO0_12
- new net IOC1: JP3.2, U$2.PIO0_13
- new net IOC2: JP3.3, U$2.PIO0_14
- new net IOC3: JP3.4, U$2.PIO0_15
- new net N$41: R48.2, U$2.GBIN0/PIO0_00
- net +3.3V: now also JP1.6
- net 12MHZ: now also R48.1, U$1.OSCI; no longer U$2.GBIN0/PIO0_00
- net AD0: now also JP4.1
- net AD1: now also JP5.1
- net AD2: now also JP4.2
- net AD3: now also JP5.2
- net AD4: now also JP4.3
- net AD5: now also JP5.3
- net ADVREF: now also JP4.4
- net GND: now also JP1.5, JP5.4, JP5.5
Other:
- note added: "Analog IOs"
- note added: "IO A"
- note added: "IO B"
- note added: "IO C"

Commit message: Started the PCB.
Parts:
- removed R32, R33, R35, R36: 0, resistor:R-US_R0603
Connections:
- removed net CTSN: R33.1
- removed net DCDN: R36.1
- removed net DSRN: R35.1
- removed net N$26: R32.2, U$1.BDBUS2
- removed net N$27: R33.2, U$1.BDBUS3
- removed net N$29: R35.2, U$1.BDBUS5
- removed net N$30: R36.2, U$1.BDBUS6
- removed net N$40: U2.VDDCORE, U2.VDDCORE_2, U2.VDDOUT, U2.VDDPLL
- removed net RTSN: R32.1
- new net VDDOUT: C43.1, C44.1, U2.VDDCORE, U2.VDDCORE_2, U2.VDDOUT, U2.VDDPLL
- net 3.3V: no longer C43.1, C44.1
Changed lines of the file:
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@@
 <setting verticaltext="up"/>
 </settings>
-<grid distance="0.1" unitdist="inch" unit="inch" style="lines" multiple="1" display="yes" altdistance="0.01" altunitdist="inch" altunit="inch"/>
+<grid distance="0.1" unitdist="inch" unit="inch" style="lines" multiple="1" display="no" altdistance="0.01" altunitdist="inch" altunit="inch"/>
 <layers>
 <layer number="1" name="Top" color="4" fill="1" visible="no" active="no"/>
@@
 <part name="R30" library="resistor" deviceset="R-US_" device="R0603" value="0"/>
 <part name="R31" library="resistor" deviceset="R-US_" device="R0603" value="0"/>
-<part name="R32" library="resistor" deviceset="R-US_" device="R0603" value="0"/>
-<part name="R33" library="resistor" deviceset="R-US_" device="R0603" value="0"/>
 <part name="R34" library="resistor" deviceset="R-US_" device="R0603" value="0"/>
-<part name="R35" library="resistor" deviceset="R-US_" device="R0603" value="0"/>
-<part name="R36" library="resistor" deviceset="R-US_" device="R0603" value="0"/>
 <part name="U2" library="Atmel_By_element14_Batch_1-00" deviceset="ATSAM3S4AA-AU" device=""/>
 <part name="U$6" library="USBC" deviceset="DX07S0" device=""/>
@@
 <text x="73.66" y="7.62" size="1.778" layer="91">Flash for FPGA</text>
 <text x="314.96" y="116.84" size="1.778" layer="91" rot="R90">For VDDin</text>
-<text x="340.36" y="127" size="1.778" layer="91">For VDDout</text>
+<text x="358.14" y="134.62" size="1.778" layer="91">For VDDout</text>
 <text x="429.26" y="40.64" size="1.778" layer="91">ADx and ADVREF still need connected to external pins</text>
 <text x="448.818" y="295.91" size="1.778" layer="91">IO A</text>
@@
 <attribute name="VALUE" x="114.554" y="106.934" size="1.778" layer="96"/>
 </instance>
-<instance part="R32" gate="G$1" x="111.76" y="104.14" smashed="yes" rot="R180">
-<attribute name="NAME" x="104.14" y="104.394" size="1.778" layer="95"/>
-<attribute name="VALUE" x="114.554" y="104.394" size="1.778" layer="96"/>
-</instance>
-<instance part="R33" gate="G$1" x="111.76" y="101.6" smashed="yes" rot="R180">
-<attribute name="NAME" x="104.14" y="101.854" size="1.778" layer="95"/>
-<attribute name="VALUE" x="114.554" y="101.854" size="1.778" layer="96"/>
-</instance>
 <instance part="R34" gate="G$1" x="111.76" y="99.06" smashed="yes" rot="R180">
 <attribute name="NAME" x="104.14" y="99.314" size="1.778" layer="95"/>
 <attribute name="VALUE" x="114.554" y="99.314" size="1.778" layer="96"/>
-</instance>
-<instance part="R35" gate="G$1" x="111.76" y="96.52" smashed="yes" rot="R180">
-<attribute name="NAME" x="104.14" y="96.774" size="1.778" layer="95"/>
-<attribute name="VALUE" x="114.554" y="96.774" size="1.778" layer="96"/>
-</instance>
-<instance part="R36" gate="G$1" x="111.76" y="93.98" smashed="yes" rot="R180">
-<attribute name="NAME" x="104.14" y="94.234" size="1.778" layer="95"/>
-<attribute name="VALUE" x="114.554" y="94.234" size="1.778" layer="96"/>
 </instance>
 <instance part="U2" gate="A" x="350.52" y="60.96"/>
@@
 </segment>
 </net>
-<net name="N$26" class="0">
-<segment>
-<pinref part="R32" gate="G$1" pin="2"/>
-<pinref part="U$1" gate="G$1" pin="BDBUS2"/>
-<wire x1="106.68" y1="104.14" x2="101.6" y2="104.14" width="0.1524" layer="91"/>
-</segment>
-</net>
-<net name="N$27" class="0">
-<segment>
-<pinref part="U$1" gate="G$1" pin="BDBUS3"/>
-<pinref part="R33" gate="G$1" pin="2"/>
-<wire x1="101.6" y1="101.6" x2="106.68" y2="101.6" width="0.1524" layer="91"/>
-</segment>
-</net>
 <net name="N$28" class="0">
 <segment>
@@
 </segment>
 </net>
-<net name="N$29" class="0">
-<segment>
-<pinref part="U$1" gate="G$1" pin="BDBUS5"/>
-<pinref part="R35" gate="G$1" pin="2"/>
-<wire x1="101.6" y1="96.52" x2="106.68" y2="96.52" width="0.1524" layer="91"/>
-</segment>
-</net>
-<net name="N$30" class="0">
-<segment>
-<pinref part="R36" gate="G$1" pin="2"/>
-<pinref part="U$1" gate="G$1" pin="BDBUS6"/>
-<wire x1="106.68" y1="93.98" x2="101.6" y2="93.98" width="0.1524" layer="91"/>
-</segment>
-</net>
-<net name="RTSN" class="0">
-<segment>
-<pinref part="R32" gate="G$1" pin="1"/>
-<wire x1="116.84" y1="104.14" x2="121.92" y2="104.14" width="0.1524" layer="91"/>
-</segment>
-</net>
-<net name="CTSN" class="0">
-<segment>
-<pinref part="R33" gate="G$1" pin="1"/>
-<wire x1="116.84" y1="101.6" x2="121.92" y2="101.6" width="0.1524" layer="91"/>
-</segment>
-</net>
 <net name="DTRN" class="0">
 <segment>
@@
 <wire x1="393.7" y1="27.94" x2="408.94" y2="27.94" width="0.1524" layer="91"/>
 <label x="401.32" y="27.94" size="1.778" layer="95"/>
-</segment>
-</net>
-<net name="DSRN" class="0">
-<segment>
-<pinref part="R35" gate="G$1" pin="1"/>
-<wire x1="116.84" y1="96.52" x2="121.92" y2="96.52" width="0.1524" layer="91"/>
-</segment>
-</net>
-<net name="DCDN" class="0">
-<segment>
-<pinref part="R36" gate="G$1" pin="1"/>
-<wire x1="116.84" y1="93.98" x2="121.92" y2="93.98" width="0.1524" layer="91"/>
 </segment>
 </net>
@@
 <segment>
 <pinref part="C42" gate="G$1" pin="1"/>
-<wire x1="317.5" y1="124.46" x2="317.5" y2="127" width="0.1524" layer="91"/>
-<wire x1="317.5" y1="127" x2="330.2" y2="127" width="0.1524" layer="91"/>
-<wire x1="330.2" y1="127" x2="340.36" y2="127" width="0.1524" layer="91"/>
-<wire x1="340.36" y1="127" x2="340.36" y2="124.46" width="0.1524" layer="91"/>
-<label x="332.74" y="137.16" size="1.778" layer="95" rot="R180"/>
-<pinref part="C43" gate="G$1" pin="1"/>
-<pinref part="C44" gate="G$1" pin="1"/>
-<wire x1="340.36" y1="127" x2="350.52" y2="127" width="0.1524" layer="91"/>
-<wire x1="350.52" y1="127" x2="350.52" y2="124.46" width="0.1524" layer="91"/>
-<junction x="340.36" y="127"/>
-<wire x1="330.2" y1="127" x2="330.2" y2="134.62" width="0.1524" layer="91"/>
-<junction x="330.2" y="127"/>
+<label x="320.04" y="137.16" size="1.778" layer="95" rot="R180"/>
+<wire x1="317.5" y1="124.46" x2="317.5" y2="134.62" width="0.1524" layer="91"/>
 </segment>
 <segment>
@@
 </segment>
 </net>
-<net name="N$40" class="0">
+<net name="VDDOUT" class="0">
 <segment>
 <pinref part="U2" gate="A" pin="VDDOUT"/>
@@
 <wire x1="297.18" y1="73.66" x2="307.34" y2="73.66" width="0.1524" layer="91"/>
 <junction x="297.18" y="76.2"/>
-</segment>
-</net>
+<label x="297.18" y="96.52" size="1.778" layer="95"/>
+<wire x1="297.18" y1="91.44" x2="297.18" y2="96.52" width="0.1524" layer="91"/>
+<junction x="297.18" y="91.44"/>
+</segment>
+<segment>
+<pinref part="C43" gate="G$1" pin="1"/>
+<wire x1="340.36" y1="124.46" x2="340.36" y2="129.54" width="0.1524" layer="91"/>
+<wire x1="340.36" y1="129.54" x2="345.44" y2="129.54" width="0.1524" layer="91"/>
+<pinref part="C44" gate="G$1" pin="1"/>
+<wire x1="345.44" y1="129.54" x2="350.52" y2="129.54" width="0.1524" layer="91"/>
+<wire x1="350.52" y1="129.54" x2="350.52" y2="124.46" width="0.1524" layer="91"/>
+<wire x1="345.44" y1="129.54" x2="345.44" y2="132.08" width="0.1524" layer="91"/>
+<junction x="345.44" y="129.54"/>
+<label x="342.9" y="132.08" size="1.778" layer="95"/>
+</segment>
+</net>

Commit message: Worked on BCP more.
Parts:
- removed R14, R15, R20, R21, R22, R23, R30, R31, R34, R48: 0, resistor:R-US_R0603
Connections:
- removed net 3.3V: C41.1, C42.1, C45.1, C46.1, C47.1, C48.1, C49.1, C50.1, C51.1, C52.1, R43.1, R45.2, R46.2, R47.2, U$7.VCC, U2.VDDIN, U2.VDDIO, U2.VDDIO_2, U2.VDDIO_3
- removed net N$11: R15.2, U$1.ACBUS7
- removed net N$12: R23.2, U$1.ACBUS0
- removed net N$13: R22.2, U$1.ACBUS1
- removed net N$14: R21.2, U$1.ACBUS2
- removed net N$17: R20.2, U$1.ACBUS4
- removed net N$24: R30.2, U$1.BDBUS0
- removed net N$25: R31.2, U$1.BDBUS1
- removed net N$28: R34.2, U$1.BDBUS4
- removed net N$41: R48.2, U$2.GBIN0/PIO0_00
- removed net N$8: R14.2, U$1.ACBUS6
- net +3.3V: now also C41.1, C42.1, C45.1, C46.1, C47.1, C48.1, C49.1, C50.1, C51.1, C52.1, R43.1, R45.2, R46.2, R47.2, U$7.VCC, U2.VDDIN, U2.VDDIO, U2.VDDIO_2, U2.VDDIO_3
- net 12MHZ: now also U$2.GBIN0/PIO0_00; no longer R48.1
- net CDONE: now also U$1.ACBUS6; no longer R14.1
- net CRESET_B: now also U$1.ACBUS7; no longer R15.1
- net DTRN: now also U$1.BDBUS4; no longer R34.1
- net MISO: now also U$1.ACBUS2; no longer R21.1
- net MOSI: now also U$1.ACBUS1; no longer R22.1
- net SCK: now also U$1.ACBUS0; no longer R23.1
- net SS: now also U$1.ACBUS4; no longer R20.1
- net URXD0: now also U$1.BDBUS0; no longer R30.1
- net UTXD0: now also U$1.BDBUS1; no longer R31.1

Commit message: Changed the diode package
Parts:
- D1: device diode:SCHOTTKY-DIODESMD -> SparkFun-DiscreteSemi:DIODE-SCHOTTKY-RB751
Changed lines of the file:
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@@
 <part name="C30" library="resistor" deviceset="C-US" device="C0603" value="0.1uF"/>
 <part name="SUPPLY12" library="supply2" deviceset="GND" device=""/>
-<part name="D1" library="diode" deviceset="SCHOTTKY-DIODE" device="SMD" value="CDBU0520"/>
 <part name="U$2" library="iCE40HX-1k" deviceset="ICE40HX1K" device=""/>
 <part name="R13" library="resistor" deviceset="R-US_" device="R0603" value="10K"/>
@@
 <part name="SUPPLY32" library="supply2" deviceset="GND" device=""/>
 <part name="SUPPLY33" library="supply2" deviceset="GND" device=""/>
+<part name="D1" library="SparkFun-DiscreteSemi" deviceset="DIODE-SCHOTTKY" device="-RB751" value="CDBU0520"/>
 </parts>
 <sheets>
@@
 <instance part="C30" gate="G$1" x="116.84" y="256.54"/>
 <instance part="SUPPLY12" gate="GND" x="162.56" y="243.84"/>
-<instance part="D1" gate="G$1" x="165.1" y="182.88" smashed="yes">
-<attribute name="NAME" x="163.83" y="184.785" size="1.778" layer="95"/>
-<attribute name="VALUE" x="160.274" y="179.451" size="1.778" layer="96"/>
-</instance>
 <instance part="U$2" gate="G$1" x="187.96" y="-30.48"/>
 <instance part="R13" gate="G$1" x="157.48" y="175.26" smashed="yes" rot="R270">
@@
 <instance part="SUPPLY32" gate="GND" x="439.42" y="195.58"/>
 <instance part="SUPPLY33" gate="GND" x="439.42" y="167.64"/>
+<instance part="D1" gate="G$1" x="165.1" y="182.88" smashed="yes">
+<attribute name="NAME" x="167.64" y="183.3626" size="1.778" layer="95"/>
+<attribute name="VALUE" x="160.02" y="179.07" size="1.778" layer="96"/>
+</instance>
 </instances>
 <busses>
@@
 </segment>
 <segment>
-<pinref part="D1" gate="G$1" pin="A"/>
 <wire x1="162.56" y1="182.88" x2="157.48" y2="182.88" width="0.1524" layer="91"/>
 <label x="154.94" y="187.96" size="1.778" layer="95"/>
@@
 <wire x1="157.48" y1="180.34" x2="157.48" y2="182.88" width="0.1524" layer="91"/>
 <junction x="157.48" y="182.88"/>
+<pinref part="D1" gate="G$1" pin="A"/>
 </segment>
 <segment>
@@
 <segment>
 <pinref part="U$2" gate="G$1" pin="VPP_2V5"/>
+<wire x1="182.88" y1="182.88" x2="167.64" y2="182.88" width="0.1524" layer="91"/>
 <pinref part="D1" gate="G$1" pin="C"/>
-<wire x1="182.88" y1="182.88" x2="167.64" y2="182.88" width="0.1524" layer="91"/>
-</segment>
-</net>
+</segment>
+</net>

Commit message: Everything but the bypass caps are on the board.
Connections:
- removed net N$18: C34.1, R24.2, R25.2, R26.2, R27.2, U$3.VCC
- net +3.3V: now also C34.1, R24.2, R25.2, R26.2, R27.2, U$3.VCC

Commit message: Added all the bypass caps to the PCB
Connections:
- net AD0: now also JP4.2; no longer JP4.1
- net AD1: now also JP5.2; no longer JP5.1
- net AD2: now also JP4.1; no longer JP4.2
- net AD3: now also JP5.1; no longer JP5.2
Changed lines of the file:
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@@
 </segment>
 <segment>
-<pinref part="JP4" gate="G$1" pin="1"/>
-<wire x1="444.5" y1="213.36" x2="434.34" y2="213.36" width="0.1524" layer="91"/>
-<label x="431.8" y="213.36" size="1.778" layer="95"/>
+<pinref part="JP4" gate="G$1" pin="2"/>
+<wire x1="444.5" y1="210.82" x2="434.34" y2="210.82" width="0.1524" layer="91"/>
+<label x="431.8" y="210.82" size="1.778" layer="95"/>
 </segment>
 </net>
@@
 </segment>
 <segment>
-<pinref part="JP5" gate="G$1" pin="1"/>
-<wire x1="444.5" y1="185.42" x2="434.34" y2="185.42" width="0.1524" layer="91"/>
-<label x="431.8" y="185.42" size="1.778" layer="95"/>
+<pinref part="JP5" gate="G$1" pin="2"/>
+<wire x1="444.5" y1="182.88" x2="434.34" y2="182.88" width="0.1524" layer="91"/>
+<label x="431.8" y="182.88" size="1.778" layer="95"/>
 </segment>
 </net>
@@
 </segment>
 <segment>
-<pinref part="JP4" gate="G$1" pin="2"/>
-<wire x1="444.5" y1="210.82" x2="434.34" y2="210.82" width="0.1524" layer="91"/>
-<label x="431.8" y="210.82" size="1.778" layer="95"/>
+<pinref part="JP4" gate="G$1" pin="1"/>
+<wire x1="444.5" y1="213.36" x2="434.34" y2="213.36" width="0.1524" layer="91"/>
+<label x="431.8" y="213.36" size="1.778" layer="95"/>
 </segment>
 </net>
@@
 </segment>
 <segment>
-<pinref part="JP5" gate="G$1" pin="2"/>
-<wire x1="444.5" y1="182.88" x2="434.34" y2="182.88" width="0.1524" layer="91"/>
-<label x="431.8" y="182.88" size="1.778" layer="95"/>
+<pinref part="JP5" gate="G$1" pin="1"/>
+<wire x1="444.5" y1="185.42" x2="434.34" y2="185.42" width="0.1524" layer="91"/>
+<label x="431.8" y="185.42" size="1.778" layer="95"/>
 </segment>
 </net>
