File: schematic/schematic.brd (EAGLE design)
At the start: 101.3 x 80 mm, 121 parts, among them U2 ATSAM3S4AA-AU

Commit message: Worked on BCP more.
Parts:
- removed R14, R15, R20, R21, R22, R23, R30, R31, R34, R48: 0, resistor:R0603
- moved C54 158.2 mm to (75.3, 18.1), turned to 270 degrees
- moved C53 143.2 mm to (65.6, 18.0), turned to 270 degrees
- moved R47 135.3 mm to (83.3, 50.2), turned to 90 degrees
- moved R46 128.1 mm to (80.9, 50.2), turned to 90 degrees
- moved R17 123.3 mm to (59.1, 22.9), turned to 90 degrees
- moved R9 103.0 mm to (22.2, 50.8), turned to 270 degrees
- moved C36 97.4 mm to (25.4, 35.6)
- moved R13 85.4 mm to (50.2, 52.1)
- moved R16 84.6 mm to (16.5, 20.3)
- moved C31 74.7 mm to (20.3, 21.6), turned to 90 degrees
- moved C22 72.3 mm to (9.53, 47.0), turned to 90 degrees
- moved C32 67.4 mm to (22.9, 21.6), turned to 90 degrees
- moved R45 64.7 mm to (8.26, 40.0), turned to 90 degrees
- moved R11 56.4 mm to (24.1, 43.2), turned to 270 degrees
- moved R12 52.9 mm to (19.7, 50.8), turned to 90 degrees
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Connections:
- removed net 3.3V: C41.1, C42.1, C45.1, C46.1, C47.1, C48.1, C49.1, C50.1, C51.1, C52.1, R43.1, R45.2, R46.2, R47.2, U$7.4, U2.13, U2.33, U2.47, U2.7
- removed net N$11: R15.2, U$1.24
- removed net N$12: R23.2, U$1.16
- removed net N$13: R22.2, U$1.17
- removed net N$14: R21.2, U$1.18
- removed net N$17: R20.2, U$1.21
- removed net N$24: R30.2, U$1.38
- removed net N$25: R31.2, U$1.39
- removed net N$28: R34.2, U$1.43
- removed net N$41: R48.2, U$2.129
- removed net N$8: R14.2, U$1.23
- net +3.3V: now also C41.1, C42.1, C45.1, C46.1, C47.1, C48.1, C49.1, C50.1, C51.1, C52.1, R43.1, R45.2, R46.2, R47.2, U$7.4, U2.13, U2.33, U2.47, U2.7
- net 12MHZ: now also U$2.129; no longer R48.1
- net CDONE: now also U$1.23; no longer R14.1
- net CRESET_B: now also U$1.24; no longer R15.1
- net DTRN: now also U$1.43; no longer R34.1
- net MISO: now also U$1.18; no longer R21.1
- net MOSI: now also U$1.17; no longer R22.1
- net SCK: now also U$1.16; no longer R23.1
- net SS: now also U$1.21; no longer R20.1
- net URXD0: now also U$1.38; no longer R30.1
- net UTXD0: now also U$1.39; no longer R31.1
Routing:
- net N$15: track 0.00 -> 11.3 mm
- net N$9: track 0.00 -> 10.9 mm
- net N$16: track 0.00 -> 6.40 mm
- net TWCK0: track 0.00 -> 5.61 mm
- net TWD0: track 0.00 -> 5.30 mm

Commit message: Changed the diode package
Parts:
- D1: device diode:SMB -> SparkFun-DiscreteSemi:SOD-523
- moved D1 154.6 mm to (-87.6, -1.27), turned to 0 degrees
Changed lines of the file:
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@@
 <element name="C8" library="resistor" package="C0603" value="0.1uF" x="-71.12" y="50.8"/>
 <element name="C9" library="resistor" package="C0603" value="0.1uF" x="-77.47" y="50.8"/>
-<element name="D1" library="diode" package="SMB" value="CDBU0520" x="58.42" y="49.53" rot="R90"/>
 <element name="JP1" library="SparkFun-Connectors" package="1X06" value="" x="96.52" y="76.2" rot="R180">
 <attribute name="PROD_ID" value="CONN-08437" x="96.52" y="76.2" size="1.778" layer="27" rot="R180" display="off"/>
@@
 <attribute name="MPN" value="ATSAM3S4AA-AU" x="81.28" y="39.37" size="1.778" layer="27" rot="R90" display="off"/>
 <attribute name="OC_FARNELL" value="1841655" x="81.28" y="39.37" size="1.778" layer="27" rot="R90" display="off"/>
+</element>
+<element name="D1" library="SparkFun-DiscreteSemi" package="SOD-523" value="CDBU0520" x="-87.63" y="-1.27">
+<attribute name="PROD_ID" value="DIO-11018" x="-87.63" y="-1.27" size="1.778" layer="27" display="off"/>
 </element>
 </elements>
@@
 <contactref element="C28" pad="1"/>
 <contactref element="C33" pad="1"/>
-<contactref element="D1" pad="A"/>
 <contactref element="R13" pad="1"/>
 <contactref element="U$2" pad="30"/>
@@
 <contactref element="U$7" pad="4"/>
 <contactref element="C41" pad="1"/>
+<contactref element="D1" pad="A"/>
 <wire x1="83.34" y1="51.06" x2="83.82" y2="76.2" width="0" layer="19" extent="1-1"/>
 <wire x1="80.94" y1="51.04" x2="83.34" y2="51.06" width="0" layer="19" extent="1-1"/>
@@
 <wire x1="85.5218" y1="36.6268" x2="81.534" y2="35.1282" width="0" layer="19" extent="1-1"/>
 <wire x1="77.89" y1="27.94" x2="81.534" y2="35.1282" width="0" layer="19" extent="1-1"/>
-<wire x1="58.42" y1="51.73" x2="80.94" y2="51.04" width="0" layer="19" extent="1-1"/>
-<wire x1="49.315" y1="52.07" x2="58.42" y2="51.73" width="0" layer="19" extent="1-1"/>
-<wire x1="42.765" y1="51.72" x2="49.315" y2="52.07" width="0" layer="19" extent="1-1"/>
+<wire x1="52.66" y1="35.23" x2="77.0382" y2="37.1094" width="0" layer="19" extent="1-1"/>
+<wire x1="52.66" y1="29.73" x2="52.66" y2="35.23" width="0" layer="19" extent="1-1"/>
+<wire x1="50.66" y1="19.73" x2="52.66" y2="29.73" width="0" layer="19" extent="1-1"/>
+<wire x1="43.16" y1="19.73" x2="50.66" y2="19.73" width="0" layer="19" extent="1-1"/>
+<wire x1="37.66" y1="19.73" x2="43.16" y2="19.73" width="0" layer="19" extent="1-1"/>
+<wire x1="31.16" y1="24.73" x2="37.66" y2="19.73" width="0" layer="19" extent="1-1"/>
+<wire x1="43.66" y1="41.23" x2="52.66" y2="35.23" width="0" layer="19" extent="1-1"/>
+<wire x1="38.66" y1="41.23" x2="43.66" y2="41.23" width="0" layer="19" extent="1-1"/>
+<wire x1="37.365" y1="48.32" x2="38.66" y2="41.23" width="0" layer="19" extent="1-1"/>
+<wire x1="34.865" y1="48.32" x2="37.365" y2="48.32" width="0" layer="19" extent="1-1"/>
+<wire x1="42.765" y1="51.72" x2="37.365" y2="48.32" width="0" layer="19" extent="1-1"/>
 <wire x1="42.765" y1="57.22" x2="42.765" y2="51.72" width="0" layer="19" extent="1-1"/>
-<wire x1="37.365" y1="48.32" x2="42.765" y2="51.72" width="0" layer="19" extent="1-1"/>
-<wire x1="34.865" y1="48.32" x2="37.365" y2="48.32" width="0" layer="19" extent="1-1"/>
+<wire x1="49.315" y1="52.07" x2="42.765" y2="51.72" width="0" layer="19" extent="1-1"/>
 <wire x1="31.465" y1="54.22" x2="34.865" y2="48.32" width="0" layer="19" extent="1-1"/>
 <wire x1="31.465" y1="57.22" x2="31.465" y2="54.22" width="0" layer="19" extent="1-1"/>
 <wire x1="36.365" y1="59.62" x2="31.465" y2="57.22" width="0" layer="19" extent="1-1"/>
-<wire x1="38.66" y1="41.23" x2="37.365" y2="48.32" width="0" layer="19" extent="1-1"/>
-<wire x1="43.66" y1="41.23" x2="38.66" y2="41.23" width="0" layer="19" extent="1-1"/>
 <wire x1="31.16" y1="36.73" x2="38.66" y2="41.23" width="0" layer="19" extent="1-1"/>
 <wire x1="24.55" y1="35.56" x2="31.16" y2="36.73" width="0" layer="19" extent="1-1"/>
@@
 <wire x1="19.685" y1="51.65" x2="12.7128" y2="47.135" width="0" layer="19" extent="1-1"/>
 <wire x1="13.755" y1="29.845" x2="16.905" y2="38.735" width="0" layer="19" extent="1-1"/>
-<wire x1="52.66" y1="35.23" x2="43.66" y2="41.23" width="0" layer="19" extent="1-1"/>
-<wire x1="52.66" y1="29.73" x2="52.66" y2="35.23" width="0" layer="19" extent="1-1"/>
-<wire x1="50.66" y1="19.73" x2="52.66" y2="29.73" width="0" layer="19" extent="1-1"/>
-<wire x1="43.16" y1="19.73" x2="50.66" y2="19.73" width="0" layer="19" extent="1-1"/>
-<wire x1="37.66" y1="19.73" x2="43.16" y2="19.73" width="0" layer="19" extent="1-1"/>
-<wire x1="31.16" y1="24.73" x2="37.66" y2="19.73" width="0" layer="19" extent="1-1"/>
 <wire x1="47.84" y1="68.58" x2="42.765" y2="57.22" width="0" layer="19" extent="1-1"/>
 <wire x1="12.28" y1="74.93" x2="19.685" y2="51.65" width="0" layer="19" extent="1-1"/>
@@
 <wire x1="-82.97" y1="71.12" x2="-82.13" y2="60.96" width="0" layer="19" extent="1-1"/>
 <wire x1="-58" y1="86.36" x2="-63.08" y2="76.2" width="0" layer="19" extent="1-1"/>
+<wire x1="-88.33" y1="-1.27" x2="-88.48" y2="55.88" width="0" layer="19" extent="1-1"/>
 </signal>
 <signal name="N$1">
@@
 <contactref element="U$2" pad="108"/>
 <contactref element="D1" pad="C"/>
-<wire x1="52.66" y1="39.23" x2="58.42" y2="47.33" width="0" layer="19" extent="1-1"/>
+<wire x1="-86.93" y1="-1.27" x2="52.66" y2="39.23" width="0" layer="19" extent="1-1"/>
 </signal>
 <signal name="N$9">

Commit message: Everything but the bypass caps are on the board.
Parts:
- moved D1 151.0 mm to (57.8, 39.4), turned to 180 degrees
- moved R28 130.9 mm to (44.5, 45.1)
- moved R24 116.1 mm to (6.99, 8.89)
- moved C39 114.5 mm to (26.7, 54.0)
- moved C38 111.3 mm to (29.2, 47.6)
- moved R19 106.4 mm to (38.7, 42.5)
- moved C37 104.7 mm to (29.2, 50.2)
- moved R18 100.8 mm to (38.7, 45.1), turned to 180 degrees
- moved C35 92.1 mm to (29.8, 59.1)
- moved R27 92.1 mm to (28.6, 7.62)
- moved R26 91.2 mm to (28.6, 5.08)
- moved C34 90.2 mm to (19.1, 10.8)
- moved C8 82.1 mm to (6.35, 23.5)
- moved R25 78.5 mm to (6.99, 6.35), turned to 180 degrees
- moved C12 72.5 mm to (15.9, 22.2)
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Connections:
- removed net N$18: C34.1, R24.2, R25.2, R26.2, R27.2, U$3.8
- net +3.3V: now also C34.1, R24.2, R25.2, R26.2, R27.2, U$3.8
Routing:
- net VBUS_5V: track 45.9 -> 34.4 mm
- net N$15: track 11.3 -> 0.00 mm
- net N$9: track 10.9 -> 0.00 mm
- net N$16: track 6.40 -> 0.00 mm
- net GND: track 23.5 -> 17.2 mm
- net N$34: track 4.08 -> 2.17 mm
- net N$33: track 4.08 -> 2.17 mm
- net N$32: track 4.08 -> 2.17 mm
- net N$31: track 4.08 -> 2.17 mm

Commit message: Added all the bypass caps to the PCB
Parts:
- moved C49 149.7 mm to (91.4, 38.1)
- moved C51 145.3 mm to (78.7, 31.1), turned to 270 degrees
- moved C48 138.0 mm to (91.4, 35.6)
- moved C6 137.0 mm to (37.5, 10.2), turned to 270 degrees
- moved C52 131.8 mm to (72.4, 35.6)
- moved C7 131.1 mm to (34.3, 10.2), turned to 270 degrees
- moved C10 130.9 mm to (40.6, 10.2), turned to 270 degrees
- moved C46 129.9 mm to (79.4, 47.0), turned to 90 degrees
- moved C14 127.9 mm to (64.8, 47.6), turned to 90 degrees
- moved C50 127.2 mm to (76.2, 47.0), turned to 90 degrees
- moved C16 123.4 mm to (64.8, 44.5), turned to 90 degrees
- moved C47 123.2 mm to (81.3, 31.1), turned to 270 degrees
- moved C23 120.0 mm to (43.8, 14.0), turned to 180 degrees
- moved C45 119.0 mm to (72.4, 38.1)
- moved C24 117.0 mm to (34.3, 14.0), turned to 180 degrees
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Connections:
- net AD0: now also JP4.2; no longer JP4.1
- net AD1: now also JP5.2; no longer JP5.1
- net AD2: now also JP4.1; no longer JP4.2
- net AD3: now also JP5.1; no longer JP5.2
Routing:
- net ADVREF: track 0.00 -> 27.0 mm
- net AD5: track 0.00 -> 25.5 mm
- net AD4: track 0.00 -> 25.0 mm
- net AD1: track 0.00 -> 19.2 mm
- net AD0: track 0.00 -> 19.2 mm, vias 0 -> 1
- net AD3: track 0.00 -> 16.7 mm
- net AD2: track 0.00 -> 12.1 mm
- net IOA3: track 0.00 -> 4.10 mm
- net VDDOUT: track 0.00 -> 4.03 mm
- net IOA2: track 0.00 -> 3.52 mm
- net N$1: track 0.00 -> 3.37 mm
- net IOA1: track 0.00 -> 2.95 mm
- net IOA0: track 0.00 -> 1.47 mm

Commit message: Removed orderThings file.
Routing:
- net FT_EEDATA: track 0.00 -> 11.2 mm
Changed lines of the file:
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@@
 <?xml version="1.0" encoding="utf-8"?>
 <!DOCTYPE eagle SYSTEM "eagle.dtd">
-<eagle version="7.3.0">
+<eagle version="7.4.0">
 <drawing>
 <settings>
@@
 <contactref element="R9" pad="1"/>
 <wire x1="22.225" y1="51.65" x2="37.115" y2="61.245" width="0" layer="19" extent="1-1"/>
-<wire x1="17.4372" y1="47.135" x2="22.225" y2="51.65" width="0" layer="19" extent="1-1"/>
+<wire x1="17.4372" y1="47.135" x2="18.56" y2="47.135" width="0.4064" layer="1"/>
+<wire x1="18.56" y1="47.135" x2="20.32" y2="48.895" width="0.4064" layer="1"/>
+<wire x1="20.32" y1="48.895" x2="23.495" y2="48.895" width="0.4064" layer="1"/>
+<wire x1="23.495" y1="48.895" x2="24.13" y2="49.53" width="0.4064" layer="1"/>
+<wire x1="24.13" y1="49.53" x2="24.13" y2="50.8" width="0.4064" layer="1"/>
+<wire x1="24.13" y1="50.8" x2="23.495" y2="51.435" width="0.4064" layer="1"/>
+<wire x1="23.495" y1="51.435" x2="22.44" y2="51.435" width="0.4064" layer="1"/>
+<wire x1="22.44" y1="51.435" x2="22.225" y2="51.65" width="0.4064" layer="1"/>
 </signal>
 <signal name="N$10">

Commit message: Made some changes to the PCB.
Parts:
- moved LED5 21.6 mm to (94.6, 38.1)
- moved LED6 21.6 mm to (94.6, 43.2)
- moved R41 21.6 mm to (88.3, 38.1)
- moved R42 21.6 mm to (88.3, 43.2)
- moved C54 18.5 mm to (63.5, 3.81)
- moved C53 16.9 mm to (74.9, 3.81)
- moved R47 13.4 mm to (82.1, 36.9)
- moved C42 13.4 mm to (73.0, 17.1)
- moved C44 13.4 mm to (83.2, 18.4)
- moved C45 13.4 mm to (71.1, 24.8)
- moved C46 13.4 mm to (78.1, 33.7)
- moved C48 13.4 mm to (90.2, 22.2)
- moved C49 13.4 mm to (90.2, 24.8)
- moved C50 13.4 mm to (74.9, 33.7)
- moved C52 13.4 mm to (71.1, 22.2)
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Connections:
- net IOC0: now also U$2.134; no longer U$2.122
- net IOC1: now also U$2.135; no longer U$2.134
- net IOC2: now also U$2.136; no longer U$2.135
- net IOC3: now also U$2.137; no longer U$2.136
Routing:
- net +1.2V: track 0.00 -> 96.6 mm, vias 0 -> 2
- net GND: track 17.2 -> 78.0 mm, vias 0 -> 5
- net IOA0: track 1.47 -> 27.9 mm
- net IOC3: track 0.00 -> 24.8 mm, vias 0 -> 1
- net LED4: track 0.00 -> 24.1 mm, vias 0 -> 2
- net IOA1: track 2.95 -> 26.3 mm
- net IOA2: track 3.52 -> 25.1 mm
- net LED3: track 0.00 -> 20.5 mm
- net IOA3: track 4.10 -> 24.2 mm
- net IOC0: track 0.00 -> 18.4 mm, vias 0 -> 1
- net IOB2: track 0.00 -> 18.4 mm, vias 0 -> 1
- net LED2: track 0.00 -> 18.4 mm
- net IOC2: track 0.00 -> 17.9 mm
- net IOB1: track 0.00 -> 17.3 mm, vias 0 -> 1
- net IOB3: track 0.00 -> 16.8 mm, vias 0 -> 1
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- added copper zone on layer 1, net +3.3V
- added copper zone on layer 16, net GND

Commit message: Added somemore traces.
Parts:
- moved JP5 66.9 mm to (70.5, 78.1), turned to 0 degrees
- moved JP4 60.3 mm to (70.5, 73.0), turned to 0 degrees
- moved C48 56.3 mm to (63.5, 71.8), turned to 90 degrees
- moved C49 55.3 mm to (61.0, 71.8), turned to 90 degrees
- moved LED6 54.9 mm to (50.8, 76.2), turned to 90 degrees
- moved LED5 54.3 mm to (55.9, 76.2), turned to 90 degrees
- moved C44 48.6 mm to (68.6, 64.8), turned to 90 degrees
- moved R42 46.0 mm to (50.8, 69.8), turned to 90 degrees
- moved R41 45.4 mm to (55.9, 69.8), turned to 90 degrees
- moved C47 45.1 mm to (69.2, 61.6), turned to 0 degrees
- moved C51 42.1 mm to (69.2, 59.1), turned to 0 degrees
- moved R47 41.7 mm to (50.1, 63.7), turned to 180 degrees
- moved U2 40.3 mm to (61.0, 61.6), turned to 180 degrees
- moved R46 38.3 mm to (50.1, 61.3), turned to 180 degrees
- moved C42 37.6 mm to (69.8, 54.6), turned to 90 degrees
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Routing:
- net GND: track 78.0 -> 163.8 mm, vias 5 -> 7
- net 12MHZ: track 0.00 -> 37.4 mm, vias 0 -> 2
- net +1.2V: track 96.6 -> 128.6 mm, vias 2 -> 5
- net +3.3V: track 1.26 -> 10.1 mm
- net N$16: track 0.00 -> 2.73 mm

Commit message: Modified PCB.
Routing:
- net GND: track 163.8 -> 171.9 mm, vias 7 -> 8
Changed lines of the file:
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@@
 <wire x1="21.59" y1="66.675" x2="23.495" y2="68.58" width="0.3048" layer="1"/>
 <wire x1="23.495" y1="68.58" x2="23.495" y2="71.755" width="0.3048" layer="1"/>
-<wire x1="55.88" y1="77.622" x2="50.8" y2="77.622" width="0" layer="19" extent="1-1"/>
-<wire x1="60.96" y1="72.605" x2="55.88" y2="77.622" width="0" layer="19" extent="1-1"/>
-<wire x1="63.5" y1="72.605" x2="60.96" y2="72.605" width="0" layer="19" extent="1-1"/>
-<wire x1="68.58" y1="65.62" x2="63.5" y2="72.605" width="0" layer="19" extent="1-1"/>
-<wire x1="70.065" y1="61.595" x2="68.58" y2="65.62" width="0" layer="19" extent="1-1"/>
-<wire x1="70.065" y1="59.055" x2="70.065" y2="61.595" width="0" layer="19" extent="1-1"/>
-<wire x1="69.85" y1="55.46" x2="70.065" y2="59.055" width="0" layer="19" extent="1-1"/>
-<wire x1="65.2018" y1="59.3344" x2="70.065" y2="59.055" width="0" layer="19" extent="1-1"/>
-<wire x1="64.77" y1="53.555" x2="69.85" y2="55.46" width="0" layer="19" extent="1-1"/>
-<wire x1="62.23" y1="53.555" x2="64.77" y2="53.555" width="0" layer="19" extent="1-1"/>
-<wire x1="56.515" y1="53.125" x2="62.23" y2="53.555" width="0" layer="19" extent="1-1"/>
-<wire x1="52.49" y1="56.515" x2="56.515" y2="53.125" width="0" layer="19" extent="1-1"/>
-<wire x1="52.49" y1="59.69" x2="52.49" y2="56.515" width="0" layer="19" extent="1-1"/>
-<wire x1="56.7182" y1="59.8424" x2="52.49" y2="59.69" width="0" layer="19" extent="1-1"/>
-<wire x1="74.93" y1="2.96" x2="70.065" y2="59.055" width="0" layer="19" extent="1-1"/>
-<wire x1="63.5" y1="2.96" x2="74.93" y2="2.96" width="0" layer="19" extent="1-1"/>
-<wire x1="78.105" y1="78.105" x2="63.5" y2="72.605" width="0" layer="19" extent="1-1"/>
+<via x="69.215" y="67.31" extent="1-16" drill="0.6" shape="octagon"/>
+<wire x1="68.58" y1="65.62" x2="68.58" y2="66.675" width="0.4064" layer="1"/>
+<wire x1="68.58" y1="66.675" x2="69.215" y2="67.31" width="0.4064" layer="1"/>
+<wire x1="70.065" y1="61.595" x2="70.065" y2="66.46" width="0.4064" layer="1"/>
+<wire x1="70.065" y1="66.46" x2="69.215" y2="67.31" width="0.4064" layer="1"/>
+<wire x1="60.96" y1="72.605" x2="63.5" y2="72.605" width="0" layer="19" extent="1-1"/>
+<wire x1="55.88" y1="77.622" x2="60.96" y2="72.605" width="0" layer="19" extent="1-1"/>
+<wire x1="50.8" y1="77.622" x2="55.88" y2="77.622" width="0" layer="19" extent="1-1"/>
+<wire x1="69.215" y1="67.31" x2="63.5" y2="72.605" width="0" layer="19" extent="1-1"/>
 <wire x1="7.86" y1="30.48" x2="8.255" y2="30.48" width="0" layer="19" extent="1-1"/>
 <wire x1="6.985" y1="30.48" x2="7.86" y2="30.48" width="0" layer="19" extent="1-1"/>
@@
 <wire x1="33.715" y1="53.345" x2="33.715" y2="54.345" width="0" layer="19" extent="1-1"/>
 <wire x1="33.715" y1="52.345" x2="33.715" y2="53.345" width="0" layer="19" extent="1-1"/>
+<wire x1="70.065" y1="59.055" x2="70.065" y2="61.595" width="0" layer="19" extent="1-1"/>
 <wire x1="30.695" y1="51.435" x2="33.715" y2="52.345" width="0" layer="19" extent="1-1"/>
 <wire x1="30.06" y1="48.895" x2="30.695" y2="51.435" width="0" layer="19" extent="1-1"/>
+<wire x1="69.85" y1="55.46" x2="70.065" y2="59.055" width="0" layer="19" extent="1-1"/>
 <wire x1="48.85" y1="23.92" x2="50.8" y2="20.74" width="0" layer="19" extent="1-1"/>
+<wire x1="65.2018" y1="59.3344" x2="70.065" y2="59.055" width="0" layer="19" extent="1-1"/>
 <wire x1="52.705" y1="27.725" x2="48.85" y2="24.42" width="0" layer="19" extent="1-1"/>
 <wire x1="56.515" y1="29.63" x2="52.705" y2="27.725" width="0" layer="19" extent="1-1"/>
 <wire x1="56.515" y1="25.185" x2="56.515" y2="29.63" width="0" layer="19" extent="1-1"/>
+<wire x1="64.77" y1="53.555" x2="69.85" y2="55.46" width="0" layer="19" extent="1-1"/>
+<wire x1="62.23" y1="53.555" x2="64.77" y2="53.555" width="0" layer="19" extent="1-1"/>
+<wire x1="64.77" y1="48.475" x2="64.77" y2="53.555" width="0" layer="19" extent="1-1"/>
+<wire x1="61.595" y1="48.475" x2="64.77" y2="48.475" width="0" layer="19" extent="1-1"/>
+<wire x1="64.77" y1="45.3" x2="64.77" y2="48.475" width="0" layer="19" extent="1-1"/>
+<wire x1="61.595" y1="45.3" x2="61.595" y2="48.475" width="0" layer="19" extent="1-1"/>
+<wire x1="56.515" y1="53.125" x2="62.23" y2="53.555" width="0" layer="19" extent="1-1"/>
+<wire x1="52.49" y1="56.515" x2="56.515" y2="53.125" width="0" layer="19" extent="1-1"/>
+<wire x1="52.49" y1="59.69" x2="52.49" y2="56.515" width="0" layer="19" extent="1-1"/>
+<wire x1="56.7182" y1="59.8424" x2="52.49" y2="59.69" width="0" layer="19" extent="1-1"/>
 <wire x1="39.615" y1="49.945" x2="33.715" y2="52.345" width="0" layer="19" extent="1-1"/>
 <wire x1="37.885" y1="45.085" x2="39.615" y2="49.945" width="0" layer="19" extent="1-1"/>
@@
 <wire x1="42.115" y1="61.245" x2="45.015" y2="58.845" width="0" layer="19" extent="1-1"/>
 <wire x1="42.965" y1="40.005" x2="36.615" y2="40.005" width="0" layer="19" extent="1-1"/>
-<wire x1="52.645" y1="41.275" x2="42.965" y2="40.005" width="0" layer="19" extent="1-1"/>
-<wire x1="52.49" y1="39.37" x2="52.645" y2="41.275" width="0" layer="19" extent="1-1"/>
-<wire x1="61.595" y1="48.475" x2="52.49" y2="39.37" width="0" layer="19" extent="1-1"/>
-<wire x1="64.77" y1="48.475" x2="61.595" y2="48.475" width="0" layer="19" extent="1-1"/>
-<wire x1="64.77" y1="45.3" x2="64.77" y2="48.475" width="0" layer="19" extent="1-1"/>
-<wire x1="61.595" y1="45.3" x2="61.595" y2="48.475" width="0" layer="19" extent="1-1"/>
+<wire x1="52.49" y1="39.37" x2="42.965" y2="40.005" width="0" layer="19" extent="1-1"/>
+<wire x1="52.645" y1="41.275" x2="52.49" y2="39.37" width="0" layer="19" extent="1-1"/>
+<wire x1="63.5" y1="2.96" x2="49.98" y2="19.92" width="0" layer="19" extent="1-1"/>
+<wire x1="74.93" y1="2.96" x2="63.5" y2="2.96" width="0" layer="19" extent="1-1"/>
 </signal>
 <signal name="N$2">
@@
 <wire x1="27.35" y1="27.42" x2="27.362" y2="27.432" width="0.3048" layer="1"/>
 <wire x1="27.362" y1="27.432" x2="28.702" y2="27.432" width="0.3048" layer="1"/>
-<wire x1="54.19" y1="59.69" x2="56.7182" y2="60.3504" width="0" layer="19" extent="1-1"/>
+<wire x1="65.2018" y1="61.849" x2="63.2206" y2="57.3532" width="0" layer="19" extent="1-1"/>
 <wire x1="68.365" y1="59.055" x2="68.365" y2="61.595" width="0" layer="19" extent="1-1"/>
+<wire x1="56.7182" y1="60.3504" x2="54.19" y2="59.69" width="0" layer="19" extent="1-1"/>
 <wire x1="48.85" y1="20.42" x2="50.8" y2="22.44" width="0" layer="19" extent="1-1"/>
 <wire x1="36.85" y1="37.42" x2="38.315" y2="40.005" width="0" layer="19" extent="1-1"/>
@@
 <wire x1="36.35" y1="15.92" x2="33.44" y2="12.7" width="0" layer="19" extent="1-1"/>
 <wire x1="48.85" y1="32.42" x2="52.705" y2="29.425" width="0" layer="19" extent="1-1"/>
-<wire x1="63.2206" y1="57.3532" x2="65.2018" y2="61.849" width="0" layer="19" extent="1-1"/>
 <wire x1="41.35" y1="15.92" x2="36.35" y2="15.92" width="0" layer="19" extent="1-1"/>
 <wire x1="44.665" y1="12.7" x2="41.35" y2="15.92" width="0" layer="19" extent="1-1"/>
@@
 <wire x1="33.715" y1="55.345" x2="28.995" y2="51.435" width="0" layer="19" extent="1-1"/>
 <wire x1="33.715" y1="57.845" x2="33.715" y2="55.345" width="0" layer="19" extent="1-1"/>
-<wire x1="39.615" y1="61.245" x2="33.715" y2="57.845" width="0" layer="19" extent="1-1"/>
-<wire x1="42.615" y1="61.245" x2="39.615" y2="61.245" width="0" layer="19" extent="1-1"/>
-<wire x1="45.015" y1="56.345" x2="42.615" y2="61.245" width="0" layer="19" extent="1-1"/>
+<wire x1="45.015" y1="56.345" x2="49.29" y2="61.255" width="0" layer="19" extent="1-1"/>
+<wire x1="42.615" y1="61.245" x2="45.015" y2="56.345" width="0" layer="19" extent="1-1"/>
+<wire x1="39.615" y1="61.245" x2="42.615" y2="61.245" width="0" layer="19" extent="1-1"/>
 </signal>
 <signal name="N$1">
@@
 <wire x1="50.99" y1="61.255" x2="50.99" y2="61.341" width="0.3048" layer="1"/>
 <wire x1="50.99" y1="61.341" x2="56.7182" y2="61.341" width="0.3048" layer="1"/>
-<wire x1="48.85" y1="18.42" x2="56.7182" y2="61.341" width="0" layer="19" extent="1-1"/>
+<wire x1="48.85" y1="18.42" x2="50.99" y2="61.255" width="0" layer="19" extent="1-1"/>
 </signal>
 <signal name="TWCK0">
@@
 <wire x1="50.97" y1="63.655" x2="51.7854" y2="62.8396" width="0.3048" layer="1"/>
 <wire x1="51.7854" y1="62.8396" x2="56.7182" y2="62.8396" width="0.3048" layer="1"/>
-<wire x1="48.85" y1="18.92" x2="56.7182" y2="62.8396" width="0" layer="19" extent="1-1"/>
+<wire x1="48.85" y1="18.92" x2="51.7854" y2="62.8396" width="0" layer="19" extent="1-1"/>
 </signal>
 <signal name="AD4">
