File: board/tinz.sch (EAGLE design)
At the start: 111 parts, among them U2 ATSAM3S4AA-AU

Commit message: Continued PCB, fixed bug.
Connections:
- removed net N$1: C22.2, U$5.VSS
- net GND: now also C22.2, U$5.VSS
Changed lines of the file:
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@@
 <part name="SUPPLY33" library="supply2" deviceset="GND" device=""/>
 <part name="D1" library="SparkFun-DiscreteSemi" deviceset="DIODE-SCHOTTKY" device="-RB751" value="CDBU0520"/>
+<part name="SUPPLY34" library="supply2" deviceset="GND" device=""/>
 </parts>
 <sheets>
@@
 <attribute name="VALUE" x="160.02" y="179.07" size="1.778" layer="96"/>
 </instance>
+<instance part="SUPPLY34" gate="GND" x="-93.98" y="81.28"/>
 </instances>
 <busses>
@@
 <pinref part="SUPPLY33" gate="GND" pin="GND"/>
 </segment>
+<segment>
+<pinref part="U$5" gate="A" pin="VSS"/>
+<wire x1="-81.28" y1="88.9" x2="-86.36" y2="88.9" width="0.1524" layer="91"/>
+<wire x1="-86.36" y1="88.9" x2="-86.36" y2="86.36" width="0.1524" layer="91"/>
+<wire x1="-86.36" y1="86.36" x2="-93.98" y2="86.36" width="0.1524" layer="91"/>
+<pinref part="C22" gate="G$1" pin="2"/>
+<wire x1="-93.98" y1="86.36" x2="-93.98" y2="88.9" width="0.1524" layer="91"/>
+<pinref part="SUPPLY34" gate="GND" pin="GND"/>
+<wire x1="-93.98" y1="83.82" x2="-93.98" y2="86.36" width="0.1524" layer="91"/>
+<junction x="-93.98" y="86.36"/>
+</segment>
 </net>
 <net name="N$2" class="0">
@@
 </segment>
 </net>
-<net name="N$1" class="0">
-<segment>
-<pinref part="U$5" gate="A" pin="VSS"/>
-<wire x1="-81.28" y1="88.9" x2="-86.36" y2="88.9" width="0.1524" layer="91"/>
-<wire x1="-86.36" y1="88.9" x2="-86.36" y2="86.36" width="0.1524" layer="91"/>
-<wire x1="-86.36" y1="86.36" x2="-93.98" y2="86.36" width="0.1524" layer="91"/>
-<pinref part="C22" gate="G$1" pin="2"/>
-<wire x1="-93.98" y1="86.36" x2="-93.98" y2="88.9" width="0.1524" layer="91"/>
-</segment>
-</net>

Commit message: Got the flash all wired up on the PCB.
Parts:
- removed R25: 10K, resistor:R-US_R0603
- added R14: 0, resistor:R-US_R0603
Connections:
- removed net N$22: R25.1, U$3.VPP/W#/DQ2
- new net N$11: R14.1, U$2.CRESET_B
- net +3.3V: now also JP2.6, JP3.6, JP4.6, JP5.6; no longer R25.2
- net CRESET_B: now also R14.2; no longer U$2.CRESET_B
- net GND: now also JP2.5, JP3.5, JP4.5
Other:
- moved on the sheet: R18, R19

Commit message: Added updated USB connector to schematic and PCB.
Connections:
- removed net DM: U$1.DM, U$6.DN1_A, U$6.DN2_B
- removed net DP: U$1.DP, U$6.DP1_A, U$6.DP2_B
- new net D_N: U$1.DM, U$6.DN
- new net D_P: U$1.DP, U$6.DP
- net GND: now also U$6.GND; no longer U$6.GND2_A, U$6.GND2_B, U$6.GND_A, U$6.GND_B
- net VBUS_5V: now also U$6.VBUS; no longer U$6.SBU2_B, U$6.VBUS2_A, U$6.VBUS2_B, U$6.VBUS_A
Changed lines of the file:
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@@
 <part name="C40" library="resistor" deviceset="C-US" device="C0603" value="10uF"/>
 <part name="U2" library="Atmel_By_element14_Batch_1-00" deviceset="ATSAM3S4AA-AU" device=""/>
-<part name="U$6" library="USBC" deviceset="DX07S0" device=""/>
 <part name="SUPPLY14" library="supply2" deviceset="GND" device=""/>
-<part name="SUPPLY20" library="supply2" deviceset="GND" device=""/>
 <part name="R37" library="resistor" deviceset="R-US_" device="R0603" value="100"/>
 <part name="LED1" library="led" deviceset="LED" device="SMT1206" value="Green"/>
@@
 <part name="SUPPLY34" library="supply2" deviceset="GND" device=""/>
 <part name="R14" library="resistor" deviceset="R-US_" device="R0603" value="0"/>
+<part name="U$6" library="USBC" deviceset="DX07S0" device=""/>
 </parts>
 <sheets>
@@
 <instance part="C40" gate="G$1" x="-10.16" y="134.62"/>
 <instance part="U2" gate="A" x="350.52" y="60.96"/>
-<instance part="U$6" gate="G$1" x="-81.28" y="40.64"/>
-<instance part="SUPPLY14" gate="GND" x="-55.88" y="17.78"/>
-<instance part="SUPPLY20" gate="GND" x="-106.68" y="17.78"/>
+<instance part="SUPPLY14" gate="GND" x="-55.88" y="-20.32"/>
 <instance part="R37" gate="G$1" x="368.3" y="215.9" smashed="yes">
 <attribute name="NAME" x="363.22" y="218.948" size="1.778" layer="95"/>
@@
 <attribute name="VALUE" x="171.958" y="164.592" size="1.778" layer="96" rot="R90"/>
 </instance>
+<instance part="U$6" gate="G$1" x="-81.28" y="-2.54"/>
 </instances>
 <busses>
@@
 </segment>
 <segment>
-<pinref part="U$6" gate="G$1" pin="GND2_B"/>
-<pinref part="SUPPLY14" gate="GND" pin="GND"/>
-<wire x1="-60.96" y1="25.4" x2="-55.88" y2="25.4" width="0.1524" layer="91"/>
-<wire x1="-55.88" y1="25.4" x2="-55.88" y2="20.32" width="0.1524" layer="91"/>
-<pinref part="U$6" gate="G$1" pin="GND_B"/>
-<wire x1="-60.96" y1="53.34" x2="-55.88" y2="53.34" width="0.1524" layer="91"/>
-<wire x1="-55.88" y1="53.34" x2="-55.88" y2="25.4" width="0.1524" layer="91"/>
-<junction x="-55.88" y="25.4"/>
-</segment>
-<segment>
-<pinref part="U$6" gate="G$1" pin="GND_A"/>
-<pinref part="SUPPLY20" gate="GND" pin="GND"/>
-<wire x1="-101.6" y1="53.34" x2="-106.68" y2="53.34" width="0.1524" layer="91"/>
-<wire x1="-106.68" y1="53.34" x2="-106.68" y2="25.4" width="0.1524" layer="91"/>
-<pinref part="U$6" gate="G$1" pin="GND2_A"/>
-<wire x1="-106.68" y1="25.4" x2="-106.68" y2="20.32" width="0.1524" layer="91"/>
-<wire x1="-101.6" y1="25.4" x2="-106.68" y2="25.4" width="0.1524" layer="91"/>
-<junction x="-106.68" y="25.4"/>
-</segment>
-<segment>
 <pinref part="LED4" gate="G$1" pin="C"/>
 <wire x1="386.08" y1="238.76" x2="391.16" y2="238.76" width="0.1524" layer="91"/>
@@
 <wire x1="444.5" y1="203.2" x2="439.42" y2="203.2" width="0.1524" layer="91"/>
 <wire x1="439.42" y1="203.2" x2="439.42" y2="198.12" width="0.1524" layer="91"/>
+</segment>
+<segment>
+<pinref part="U$6" gate="G$1" pin="GND"/>
+<wire x1="-60.96" y1="10.16" x2="-55.88" y2="10.16" width="0.1524" layer="91"/>
+<wire x1="-55.88" y1="10.16" x2="-55.88" y2="-17.78" width="0.1524" layer="91"/>
+<pinref part="SUPPLY14" gate="GND" pin="GND"/>
 </segment>
 </net>
@@
 </segment>
 <segment>
-<pinref part="U$6" gate="G$1" pin="VBUS2_B"/>
-<wire x1="-60.96" y1="33.02" x2="-53.34" y2="33.02" width="0.1524" layer="91"/>
-<wire x1="-53.34" y1="33.02" x2="-53.34" y2="43.18" width="0.1524" layer="91"/>
-<pinref part="U$6" gate="G$1" pin="SBU2_B"/>
-<wire x1="-53.34" y1="43.18" x2="-60.96" y2="43.18" width="0.1524" layer="91"/>
-<wire x1="-53.34" y1="43.18" x2="-53.34" y2="60.96" width="0.1524" layer="91"/>
-<junction x="-53.34" y="43.18"/>
-<pinref part="U$6" gate="G$1" pin="VBUS2_A"/>
-<wire x1="-101.6" y1="33.02" x2="-111.76" y2="33.02" width="0.1524" layer="91"/>
-<wire x1="-111.76" y1="33.02" x2="-111.76" y2="45.72" width="0.1524" layer="91"/>
-<pinref part="U$6" gate="G$1" pin="VBUS_A"/>
-<wire x1="-111.76" y1="45.72" x2="-101.6" y2="45.72" width="0.1524" layer="91"/>
-<wire x1="-111.76" y1="45.72" x2="-111.76" y2="60.96" width="0.1524" layer="91"/>
-<junction x="-111.76" y="45.72"/>
-<wire x1="-53.34" y1="60.96" x2="-88.9" y2="60.96" width="0.1524" layer="91"/>
-<wire x1="-88.9" y1="60.96" x2="-111.76" y2="60.96" width="0.1524" layer="91"/>
-<wire x1="-88.9" y1="60.96" x2="-88.9" y2="66.04" width="0.1524" layer="91"/>
-<junction x="-88.9" y="60.96"/>
-<label x="-93.98" y="66.04" size="1.778" layer="95"/>
-</segment>
-<segment>
 <pinref part="R44" gate="G$1" pin="1"/>
 <wire x1="-152.4" y1="81.28" x2="-165.1" y2="81.28" width="0.1524" layer="91"/>
 <label x="-165.1" y="81.28" size="1.778" layer="95"/>
+</segment>
+<segment>
+<pinref part="U$6" gate="G$1" pin="VBUS"/>
+<wire x1="-60.96" y1="7.62" x2="-48.26" y2="7.62" width="0.1524" layer="91"/>
+<label x="-48.26" y="7.62" size="1.778" layer="95"/>
 </segment>
 </net>
@@
 </segment>
 </net>
-<net name="DM" class="0">
-<segment>
-<pinref part="U$6" gate="G$1" pin="DN1_A"/>
-<wire x1="-101.6" y1="38.1" x2="-124.46" y2="38.1" width="0.1524" layer="91"/>
-<label x="-124.46" y="38.1" size="1.778" layer="95"/>
-</segment>
-<segment>
-<pinref part="U$6" gate="G$1" pin="DN2_B"/>
-<wire x1="-60.96" y1="40.64" x2="-43.18" y2="40.64" width="0.1524" layer="91"/>
-<label x="-45.72" y="40.64" size="1.778" layer="95"/>
-</segment>
-<segment>
-<pinref part="U$1" gate="G$1" pin="DM"/>
-<wire x1="33.02" y1="137.16" x2="25.4" y2="137.16" width="0.1524" layer="91"/>
-<label x="25.4" y="137.16" size="1.778" layer="95"/>
-</segment>
-</net>
-<net name="DP" class="0">
-<segment>
-<pinref part="U$6" gate="G$1" pin="DP1_A"/>
-<wire x1="-101.6" y1="40.64" x2="-124.46" y2="40.64" width="0.1524" layer="91"/>
-<label x="-124.46" y="40.64" size="1.778" layer="95"/>
-</segment>
-<segment>
-<pinref part="U$6" gate="G$1" pin="DP2_B"/>
-<wire x1="-60.96" y1="38.1" x2="-43.18" y2="38.1" width="0.1524" layer="91"/>
-<label x="-45.72" y="38.1" size="1.778" layer="95"/>
-</segment>
-<segment>
-<pinref part="U$1" gate="G$1" pin="DP"/>
-<wire x1="33.02" y1="134.62" x2="25.4" y2="134.62" width="0.1524" layer="91"/>
-<label x="25.4" y="134.62" size="1.778" layer="95"/>
-</segment>
-</net>
 <net name="URXD0" class="0">
 <segment>
@@
 </segment>
 </net>
+<net name="D_N" class="0">
+<segment>
+<pinref part="U$6" gate="G$1" pin="DN"/>
+<wire x1="-60.96" y1="0" x2="-48.26" y2="0" width="0.1524" layer="91"/>
+<label x="-48.26" y="0" size="1.778" layer="95"/>
+</segment>
+<segment>
+<pinref part="U$1" gate="G$1" pin="DM"/>
+<wire x1="33.02" y1="137.16" x2="25.4" y2="137.16" width="0.1524" layer="91"/>
+<label x="25.4" y="137.16" size="1.778" layer="95"/>
+</segment>
+</net>
+<net name="D_P" class="0">
+<segment>
+<pinref part="U$6" gate="G$1" pin="DP"/>
+<wire x1="-60.96" y1="-2.54" x2="-48.26" y2="-2.54" width="0.1524" layer="91"/>
+<label x="-48.26" y="-2.54" size="1.778" layer="95"/>
+</segment>
+<segment>
+<pinref part="U$1" gate="G$1" pin="DP"/>
+<wire x1="33.02" y1="134.62" x2="25.4" y2="134.62" width="0.1524" layer="91"/>
+<label x="25.4" y="134.62" size="1.778" layer="95"/>
+</segment>
+</net>
 </nets>
 </sheet>
 </sheets>
+<errors>
+</errors>
 </schematic>
 </drawing>
