File: board/tinz.sch (EAGLE design)
At the start: 111 parts, among them U2 ATSAM3S4AA-AU

Commit message: Untwisted most of the wires between the MCU and GPIO.
Connections:
- net GPIO0: now also U$2.PIO3_17/DP10B; no longer U$2.PIO3_11/DP04B
- net GPIO1: now also U$2.PIO3_16/DP10A; no longer U$2.PIO3_12/DP07A
- net GPIO2: now also U$2.PIO3_15/DP09B; no longer U$2.GBIN7/PIO3_01/DP07B
- net GPIO3: now also U$2.PIO3_14/DP09A; no longer U$2.GBIN6/PIO3_00/DP08A
- net GPIO5: now also U$2.PIO3_11/DP04B; no longer U$2.PIO3_14/DP09A
- net GPIO6: now also U$2.PIO3_12/DP07A; no longer U$2.PIO3_15/DP09B
- net GPIO7: now also U$2.GBIN6/PIO3_00/DP08A; no longer U$2.PIO3_16/DP10A
- net GPIO8: now also U$2.GBIN7/PIO3_01/DP07B; no longer U$2.PIO3_17/DP10B
- net M_MISO: now also U$2.PIO2_12; no longer U$2.PIO2_13
- net M_MOSI: now also U$2.PIO2_13; no longer U$2.PIO2_12
- net TWCK0: now also U$2.PIO3_03/DP00B; no longer U$2.PIO3_04/DP01A
- net TWD0: now also U$2.PIO3_04/DP01A; no longer U$2.PIO3_03/DP00B
Changed lines of the file:
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@@
 <net name="M_MOSI" class="0">
-<segment>
-<pinref part="U$2" gate="G$1" pin="PIO2_12"/>
-<wire x1="233.68" y1="60.96" x2="256.54" y2="60.96" width="0.1524" layer="91"/>
-<label x="241.3" y="60.96" size="1.778" layer="95"/>
-</segment>
 <segment>
 <pinref part="U2" gate="A" pin="PA13/PGMD1"/>
@@
 <label x="403.86" y="53.34" size="1.778" layer="95"/>
 </segment>
+<segment>
+<pinref part="U$2" gate="G$1" pin="PIO2_13"/>
+<wire x1="233.68" y1="58.42" x2="256.54" y2="58.42" width="0.1524" layer="91"/>
+<label x="246.38" y="58.42" size="1.778" layer="95"/>
+</segment>
 </net>
 <net name="SPI_NPCS0" class="0">
@@
 <net name="M_MISO" class="0">
 <segment>
-<pinref part="U$2" gate="G$1" pin="PIO2_13"/>
-<wire x1="233.68" y1="58.42" x2="256.54" y2="58.42" width="0.1524" layer="91"/>
-<label x="241.3" y="58.42" size="1.778" layer="95"/>
-</segment>
-<segment>
 <pinref part="U2" gate="A" pin="PA12/PGMD0"/>
 <wire x1="393.7" y1="55.88" x2="414.02" y2="55.88" width="0.1524" layer="91"/>
 <label x="403.86" y="55.88" size="1.778" layer="95"/>
 </segment>
+<segment>
+<pinref part="U$2" gate="G$1" pin="PIO2_12"/>
+<wire x1="233.68" y1="60.96" x2="256.54" y2="60.96" width="0.1524" layer="91"/>
+<label x="246.38" y="60.96" size="1.778" layer="95"/>
+</segment>
 </net>
 <net name="URXD1" class="0">
@@
 </segment>
 <segment>
-<pinref part="U$2" gate="G$1" pin="PIO3_16/DP10A"/>
-<wire x1="233.68" y1="-5.08" x2="246.38" y2="-5.08" width="0.1524" layer="91"/>
-<label x="238.76" y="-5.08" size="1.778" layer="95"/>
+<pinref part="U$2" gate="G$1" pin="GBIN6/PIO3_00/DP08A"/>
+<wire x1="233.68" y1="35.56" x2="246.38" y2="35.56" width="0.1524" layer="91"/>
+<label x="238.76" y="35.56" size="1.778" layer="95"/>
 </segment>
 </net>
@@
 </segment>
 <segment>
-<pinref part="U$2" gate="G$1" pin="PIO3_17/DP10B"/>
-<wire x1="233.68" y1="-7.62" x2="246.38" y2="-7.62" width="0.1524" layer="91"/>
-<label x="238.76" y="-7.62" size="1.778" layer="95"/>
+<pinref part="U$2" gate="G$1" pin="GBIN7/PIO3_01/DP07B"/>
+<wire x1="233.68" y1="33.02" x2="246.38" y2="33.02" width="0.1524" layer="91"/>
+<label x="238.76" y="33.02" size="1.778" layer="95"/>
 </segment>
 </net>
@@
 </segment>
 <segment>
-<pinref part="U$2" gate="G$1" pin="PIO3_03/DP00B"/>
-<wire x1="233.68" y1="27.94" x2="246.38" y2="27.94" width="0.1524" layer="91"/>
-<label x="238.76" y="27.94" size="1.778" layer="95"/>
+<pinref part="U$2" gate="G$1" pin="PIO3_04/DP01A"/>
+<wire x1="233.68" y1="25.4" x2="246.38" y2="25.4" width="0.1524" layer="91"/>
+<label x="238.76" y="25.4" size="1.778" layer="95"/>
 </segment>
 </net>
@@
 </segment>
 <segment>
-<pinref part="U$2" gate="G$1" pin="PIO3_04/DP01A"/>
-<wire x1="233.68" y1="25.4" x2="246.38" y2="25.4" width="0.1524" layer="91"/>
-<label x="238.76" y="25.4" size="1.778" layer="95"/>
+<pinref part="U$2" gate="G$1" pin="PIO3_03/DP00B"/>
+<wire x1="233.68" y1="27.94" x2="246.38" y2="27.94" width="0.1524" layer="91"/>
+<label x="238.76" y="27.94" size="1.778" layer="95"/>
 </segment>
 </net>
@@
 </segment>
 <segment>
+<pinref part="U$2" gate="G$1" pin="PIO3_17/DP10B"/>
+<wire x1="233.68" y1="-7.62" x2="246.38" y2="-7.62" width="0.1524" layer="91"/>
+<label x="238.76" y="-7.62" size="1.778" layer="95"/>
+</segment>
+</net>
+<net name="GPIO1" class="0">
+<segment>
+<pinref part="U2" gate="A" pin="PA1/PGMEN1"/>
+<wire x1="393.7" y1="83.82" x2="406.4" y2="83.82" width="0.1524" layer="91"/>
+<label x="398.78" y="83.82" size="1.778" layer="95"/>
+</segment>
+<segment>
+<pinref part="U$2" gate="G$1" pin="PIO3_16/DP10A"/>
+<wire x1="233.68" y1="-5.08" x2="246.38" y2="-5.08" width="0.1524" layer="91"/>
+<label x="238.76" y="-5.08" size="1.778" layer="95"/>
+</segment>
+</net>
+<net name="GPIO2" class="0">
+<segment>
+<pinref part="U2" gate="A" pin="PA2/PGMEN2"/>
+<wire x1="393.7" y1="81.28" x2="406.4" y2="81.28" width="0.1524" layer="91"/>
+<label x="398.78" y="81.28" size="1.778" layer="95"/>
+</segment>
+<segment>
+<pinref part="U$2" gate="G$1" pin="PIO3_15/DP09B"/>
+<wire x1="233.68" y1="-2.54" x2="246.38" y2="-2.54" width="0.1524" layer="91"/>
+<label x="238.76" y="-2.54" size="1.778" layer="95"/>
+</segment>
+</net>
+<net name="GPIO3" class="0">
+<segment>
+<pinref part="U2" gate="A" pin="PA6/PGMNOE"/>
+<wire x1="393.7" y1="71.12" x2="408.94" y2="71.12" width="0.1524" layer="91"/>
+<label x="401.32" y="71.12" size="1.778" layer="95"/>
+</segment>
+<segment>
+<pinref part="U$2" gate="G$1" pin="PIO3_14/DP09A"/>
+<wire x1="233.68" y1="0" x2="246.38" y2="0" width="0.1524" layer="91"/>
+<label x="238.76" y="0" size="1.778" layer="95"/>
+</segment>
+</net>
+<net name="GPIO4" class="0">
+<segment>
+<pinref part="U2" gate="A" pin="PA8/XOUT32/PGMM0"/>
+<wire x1="393.7" y1="66.04" x2="408.94" y2="66.04" width="0.1524" layer="91"/>
+<label x="401.32" y="66.04" size="1.778" layer="95"/>
+</segment>
+<segment>
+<pinref part="U$2" gate="G$1" pin="PIO3_13/DP08B"/>
+<wire x1="233.68" y1="2.54" x2="246.38" y2="2.54" width="0.1524" layer="91"/>
+<label x="238.76" y="2.54" size="1.778" layer="95"/>
+</segment>
+</net>
+<net name="GPIO5" class="0">
+<segment>
+<pinref part="U2" gate="A" pin="PA15/PGMD3"/>
+<wire x1="393.7" y1="48.26" x2="411.48" y2="48.26" width="0.1524" layer="91"/>
+<label x="403.86" y="48.26" size="1.778" layer="95"/>
+</segment>
+<segment>
 <pinref part="U$2" gate="G$1" pin="PIO3_11/DP04B"/>
 <wire x1="233.68" y1="7.62" x2="246.38" y2="7.62" width="0.1524" layer="91"/>
@@
 </segment>
 </net>
-<net name="GPIO1" class="0">
-<segment>
-<pinref part="U2" gate="A" pin="PA1/PGMEN1"/>
-<wire x1="393.7" y1="83.82" x2="406.4" y2="83.82" width="0.1524" layer="91"/>
-<label x="398.78" y="83.82" size="1.778" layer="95"/>
+<net name="GPIO6" class="0">
+<segment>
+<pinref part="U2" gate="A" pin="PA16/PGMD4"/>
+<wire x1="393.7" y1="45.72" x2="411.48" y2="45.72" width="0.1524" layer="91"/>
+<label x="403.86" y="45.72" size="1.778" layer="95"/>
 </segment>
 <segment>
@@
 </segment>
 </net>
-<net name="GPIO2" class="0">
-<segment>
-<pinref part="U2" gate="A" pin="PA2/PGMEN2"/>
-<wire x1="393.7" y1="81.28" x2="406.4" y2="81.28" width="0.1524" layer="91"/>
-<label x="398.78" y="81.28" size="1.778" layer="95"/>
-</segment>
-<segment>
-<pinref part="U$2" gate="G$1" pin="GBIN7/PIO3_01/DP07B"/>
-<wire x1="233.68" y1="33.02" x2="246.38" y2="33.02" width="0.1524" layer="91"/>
-<label x="238.76" y="33.02" size="1.778" layer="95"/>
-</segment>
-</net>
-<net name="GPIO3" class="0">
-<segment>
-<pinref part="U2" gate="A" pin="PA6/PGMNOE"/>
-<wire x1="393.7" y1="71.12" x2="408.94" y2="71.12" width="0.1524" layer="91"/>
-<label x="401.32" y="71.12" size="1.778" layer="95"/>
-</segment>
-<segment>
-<pinref part="U$2" gate="G$1" pin="GBIN6/PIO3_00/DP08A"/>
-<wire x1="233.68" y1="35.56" x2="246.38" y2="35.56" width="0.1524" layer="91"/>
-<label x="238.76" y="35.56" size="1.778" layer="95"/>
-</segment>
-</net>
-<net name="GPIO4" class="0">
-<segment>
-<pinref part="U2" gate="A" pin="PA8/XOUT32/PGMM0"/>
-<wire x1="393.7" y1="66.04" x2="408.94" y2="66.04" width="0.1524" layer="91"/>
-<label x="401.32" y="66.04" size="1.778" layer="95"/>
-</segment>
-<segment>
-<pinref part="U$2" gate="G$1" pin="PIO3_13/DP08B"/>
-<wire x1="233.68" y1="2.54" x2="246.38" y2="2.54" width="0.1524" layer="91"/>
-<label x="238.76" y="2.54" size="1.778" layer="95"/>
-</segment>
-</net>
-<net name="GPIO5" class="0">
-<segment>
-<pinref part="U2" gate="A" pin="PA15/PGMD3"/>
-<wire x1="393.7" y1="48.26" x2="411.48" y2="48.26" width="0.1524" layer="91"/>
-<label x="403.86" y="48.26" size="1.778" layer="95"/>
-</segment>
-<segment>
-<pinref part="U$2" gate="G$1" pin="PIO3_14/DP09A"/>
-<wire x1="233.68" y1="0" x2="246.38" y2="0" width="0.1524" layer="91"/>
-<label x="238.76" y="0" size="1.778" layer="95"/>
-</segment>
-</net>
-<net name="GPIO6" class="0">
-<segment>
-<pinref part="U2" gate="A" pin="PA16/PGMD4"/>
-<wire x1="393.7" y1="45.72" x2="411.48" y2="45.72" width="0.1524" layer="91"/>
-<label x="403.86" y="45.72" size="1.778" layer="95"/>
-</segment>
-<segment>
-<pinref part="U$2" gate="G$1" pin="PIO3_15/DP09B"/>
-<wire x1="233.68" y1="-2.54" x2="246.38" y2="-2.54" width="0.1524" layer="91"/>
-<label x="238.76" y="-2.54" size="1.778" layer="95"/>
-</segment>
-</net>

Commit message: Ran the TWI and UART traces
Connections:
- net TWCK0: now also U$2.PIO2_06; no longer U$2.PIO3_03/DP00B
- net TWD0: now also U$2.PIO2_05; no longer U$2.PIO3_04/DP01A
Changed lines of the file:
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@@
 </segment>
 <segment>
-<pinref part="U$2" gate="G$1" pin="PIO3_04/DP01A"/>
-<wire x1="233.68" y1="25.4" x2="246.38" y2="25.4" width="0.1524" layer="91"/>
-<label x="238.76" y="25.4" size="1.778" layer="95"/>
+<pinref part="U$2" gate="G$1" pin="PIO2_05"/>
+<wire x1="233.68" y1="78.74" x2="256.54" y2="78.74" width="0.1524" layer="91"/>
 </segment>
 </net>
@@
 </segment>
 <segment>
-<pinref part="U$2" gate="G$1" pin="PIO3_03/DP00B"/>
-<wire x1="233.68" y1="27.94" x2="246.38" y2="27.94" width="0.1524" layer="91"/>
-<label x="238.76" y="27.94" size="1.778" layer="95"/>
+<pinref part="U$2" gate="G$1" pin="PIO2_06"/>
+<wire x1="233.68" y1="76.2" x2="256.54" y2="76.2" width="0.1524" layer="91"/>
 </segment>
 </net>

Commit message: Some more wires added.
Parts:
- removed R14: 0, resistor:R-US_R0603
Connections:
- removed net N$11: R14.1, U$2.CRESET_B
- net CRESET_B: now also U$2.CRESET_B; no longer R14.2
- net GPIO0: now also U2.PA1/PGMEN1; no longer U2.PA0/PGMEN0
- net GPIO1: now also U2.PA0/PGMEN0; no longer U2.PA1/PGMEN1
Other:
- note added: "dont include"
Changed lines of the file:
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@@
 <part name="D1" library="SparkFun-DiscreteSemi" deviceset="DIODE-SCHOTTKY" device="-RB751" value="CDBU0520"/>
 <part name="SUPPLY34" library="supply2" deviceset="GND" device=""/>
-<part name="R14" library="resistor" deviceset="R-US_" device="R0603" value="0"/>
 <part name="U$6" library="USBC" deviceset="DX07S0" device=""/>
 </parts>
@@
 <text x="448.818" y="242.57" size="1.778" layer="91">IO C</text>
 <text x="444.5" y="190.5" size="1.778" layer="91">Analog IOs</text>
+<text x="165.862" y="148.59" size="1.778" layer="91">dont include</text>
 </plain>
 <instances>
@@
 </instance>
 <instance part="SUPPLY34" gate="GND" x="-93.98" y="81.28"/>
-<instance part="R14" gate="G$1" x="172.72" y="167.64" smashed="yes" rot="R180">
-<attribute name="NAME" x="175.26" y="162.052" size="1.778" layer="95" rot="R90"/>
-<attribute name="VALUE" x="171.958" y="164.592" size="1.778" layer="96" rot="R90"/>
-</instance>
 <instance part="U$6" gate="G$1" x="-81.28" y="-2.54"/>
 </instances>
@@
 <pinref part="R18" gate="G$1" pin="1"/>
 <wire x1="165.1" y1="152.4" x2="165.1" y2="149.86" width="0.1524" layer="91"/>
-<pinref part="R14" gate="G$1" pin="2"/>
-<wire x1="167.64" y1="167.64" x2="165.1" y2="167.64" width="0.1524" layer="91"/>
 <wire x1="165.1" y1="167.64" x2="165.1" y2="152.4" width="0.1524" layer="91"/>
 <junction x="165.1" y="152.4"/>
@@
 <junction x="165.1" y="167.64"/>
 <label x="139.192" y="167.132" size="1.778" layer="95"/>
+<pinref part="U$2" gate="G$1" pin="CRESET_B"/>
+<wire x1="165.1" y1="167.64" x2="182.88" y2="167.64" width="0.1524" layer="91"/>
 </segment>
 </net>
@@
 <net name="GPIO0" class="0">
 <segment>
+<pinref part="U$2" gate="G$1" pin="PIO3_17/DP10B"/>
+<wire x1="233.68" y1="-7.62" x2="246.38" y2="-7.62" width="0.1524" layer="91"/>
+<label x="238.76" y="-7.62" size="1.778" layer="95"/>
+</segment>
+<segment>
+<pinref part="U2" gate="A" pin="PA1/PGMEN1"/>
+<wire x1="393.7" y1="83.82" x2="406.4" y2="83.82" width="0.1524" layer="91"/>
+<label x="398.78" y="83.82" size="1.778" layer="95"/>
+</segment>
+</net>
+<net name="GPIO1" class="0">
+<segment>
+<pinref part="U$2" gate="G$1" pin="PIO3_16/DP10A"/>
+<wire x1="233.68" y1="-5.08" x2="246.38" y2="-5.08" width="0.1524" layer="91"/>
+<label x="238.76" y="-5.08" size="1.778" layer="95"/>
+</segment>
+<segment>
 <pinref part="U2" gate="A" pin="PA0/PGMEN0"/>
 <wire x1="393.7" y1="86.36" x2="406.4" y2="86.36" width="0.1524" layer="91"/>
 <label x="398.78" y="86.36" size="1.778" layer="95"/>
 </segment>
-<segment>
-<pinref part="U$2" gate="G$1" pin="PIO3_17/DP10B"/>
-<wire x1="233.68" y1="-7.62" x2="246.38" y2="-7.62" width="0.1524" layer="91"/>
-<label x="238.76" y="-7.62" size="1.778" layer="95"/>
-</segment>
-</net>
-<net name="GPIO1" class="0">
-<segment>
-<pinref part="U2" gate="A" pin="PA1/PGMEN1"/>
-<wire x1="393.7" y1="83.82" x2="406.4" y2="83.82" width="0.1524" layer="91"/>
-<label x="398.78" y="83.82" size="1.778" layer="95"/>
-</segment>
-<segment>
-<pinref part="U$2" gate="G$1" pin="PIO3_16/DP10A"/>
-<wire x1="233.68" y1="-5.08" x2="246.38" y2="-5.08" width="0.1524" layer="91"/>
-<label x="238.76" y="-5.08" size="1.778" layer="95"/>
-</segment>
 </net>
 <net name="GPIO2" class="0">
@@
 </segment>
 </net>
-<net name="N$11" class="0">
-<segment>
-<pinref part="U$2" gate="G$1" pin="CRESET_B"/>
-<pinref part="R14" gate="G$1" pin="1"/>
-<wire x1="182.88" y1="167.64" x2="177.8" y2="167.64" width="0.1524" layer="91"/>
-</segment>
-</net>

Commit message: Added the ecx crystal oscillator.
Parts:
- removed Q1: (no value), crystal:CRYSTALHC49UP
- added U$8: ECO32, ecx32:ECO32
Connections:
- removed net GPIO2: U$2.PIO3_15/DP09B, U2.PA2/PGMEN2
- removed net GPIO3: U$2.PIO3_14/DP09A, U2.PA6/PGMNOE
- removed net GPIO4: U$2.PIO3_13/DP08B, U2.PA8/XOUT32/PGMM0
- removed net GPIO5: U$2.PIO3_11/DP04B, U2.PA15/PGMD3
- removed net GPIO6: U$2.PIO3_12/DP07A, U2.PA16/PGMD4
- removed net GPIO7: U$2.GBIN6/PIO3_00/DP08A, U2.DDM/PB10
- removed net GPIO8: U$2.GBIN7/PIO3_01/DP07B, U2.DDP/PB11
- net GND: now also U$8.GND
- net XIN: now also U$8.IO2; no longer Q1.2
- net XOUT: now also U$8.IO1; no longer Q1.1
Changed lines of the file:
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@@
 <part name="C51" library="resistor" deviceset="C-US" device="C0603" value="10uF"/>
 <part name="C52" library="resistor" deviceset="C-US" device="C0603" value="0.1uF"/>
-<part name="Q1" library="crystal" deviceset="CRYSTAL" device="HC49UP"/>
 <part name="C53" library="resistor" deviceset="C-US" device="C0603" value="56pF"/>
 <part name="C54" library="resistor" deviceset="C-US" device="C0603" value="56pF"/>
@@
 <part name="SUPPLY34" library="supply2" deviceset="GND" device=""/>
 <part name="U$6" library="USBC" deviceset="DX07S0" device=""/>
+<part name="SUPPLY20" library="supply2" deviceset="GND" device=""/>
+<part name="U$8" library="ecx32" deviceset="ECO32" device=""/>
 </parts>
 <sheets>
@@
 <instance part="C51" gate="G$1" x="406.4" y="137.16"/>
 <instance part="C52" gate="G$1" x="482.6" y="137.16"/>
-<instance part="Q1" gate="G$1" x="467.36" y="83.82" rot="R180"/>
 <instance part="C53" gate="G$1" x="457.2" y="73.66"/>
 <instance part="C54" gate="G$1" x="477.52" y="73.66"/>
@@
 <instance part="SUPPLY34" gate="GND" x="-93.98" y="81.28"/>
 <instance part="U$6" gate="G$1" x="-81.28" y="-2.54"/>
+<instance part="SUPPLY20" gate="GND" x="467.36" y="73.66"/>
+<instance part="U$8" gate="G$1" x="467.36" y="83.82" smashed="yes" rot="R180">
+<attribute name="NAME" x="471.932" y="89.154" size="1.778" layer="95" rot="R180"/>
+<attribute name="VALUE" x="472.44" y="91.44" size="1.778" layer="96" rot="R180"/>
+</instance>
 </instances>
 <busses>
@@
 <pinref part="SUPPLY14" gate="GND" pin="GND"/>
 </segment>
+<segment>
+<pinref part="SUPPLY20" gate="GND" pin="GND"/>
+<wire x1="467.36" y1="76.2" x2="467.36" y2="78.74" width="0.1524" layer="91"/>
+<pinref part="U$8" gate="G$1" pin="GND"/>
+</segment>
 </net>
 <net name="N$2" class="0">
@@
 <net name="XIN" class="0">
 <segment>
-<pinref part="Q1" gate="G$1" pin="2"/>
 <wire x1="457.2" y1="83.82" x2="464.82" y2="83.82" width="0.1524" layer="91"/>
 <pinref part="C53" gate="G$1" pin="1"/>
@@
 <junction x="457.2" y="83.82"/>
 <label x="454.66" y="91.44" size="1.778" layer="95"/>
+<pinref part="U$8" gate="G$1" pin="IO2"/>
 </segment>
 <segment>
@@
 <net name="XOUT" class="0">
 <segment>
-<pinref part="Q1" gate="G$1" pin="1"/>
 <wire x1="477.52" y1="83.82" x2="469.9" y2="83.82" width="0.1524" layer="91"/>
 <pinref part="C54" gate="G$1" pin="1"/>
@@
 <junction x="477.52" y="83.82"/>
 <label x="474.98" y="91.44" size="1.778" layer="95"/>
+<pinref part="U$8" gate="G$1" pin="IO1"/>
 </segment>
 <segment>
@@
 <wire x1="307.34" y1="50.8" x2="297.18" y2="50.8" width="0.1524" layer="91"/>
 <label x="297.18" y="50.8" size="1.778" layer="95"/>
-</segment>
-</net>
-<net name="GPIO7" class="0">
-<segment>
-<pinref part="U2" gate="A" pin="DDM/PB10"/>
-<wire x1="307.34" y1="33.02" x2="297.18" y2="33.02" width="0.1524" layer="91"/>
-<label x="297.18" y="33.02" size="1.778" layer="95"/>
-</segment>
-<segment>
-<pinref part="U$2" gate="G$1" pin="GBIN6/PIO3_00/DP08A"/>
-<wire x1="233.68" y1="35.56" x2="246.38" y2="35.56" width="0.1524" layer="91"/>
-<label x="238.76" y="35.56" size="1.778" layer="95"/>
-</segment>
-</net>
-<net name="GPIO8" class="0">
-<segment>
-<pinref part="U2" gate="A" pin="DDP/PB11"/>
-<wire x1="393.7" y1="30.48" x2="408.94" y2="30.48" width="0.1524" layer="91"/>
-<label x="401.32" y="30.48" size="1.778" layer="95"/>
-</segment>
-<segment>
-<pinref part="U$2" gate="G$1" pin="GBIN7/PIO3_01/DP07B"/>
-<wire x1="233.68" y1="33.02" x2="246.38" y2="33.02" width="0.1524" layer="91"/>
-<label x="238.76" y="33.02" size="1.778" layer="95"/>
 </segment>
 </net>
@@
 </segment>
 </net>
-<net name="GPIO2" class="0">
-<segment>
-<pinref part="U2" gate="A" pin="PA2/PGMEN2"/>
-<wire x1="393.7" y1="81.28" x2="406.4" y2="81.28" width="0.1524" layer="91"/>
-<label x="398.78" y="81.28" size="1.778" layer="95"/>
-</segment>
-<segment>
-<pinref part="U$2" gate="G$1" pin="PIO3_15/DP09B"/>
-<wire x1="233.68" y1="-2.54" x2="246.38" y2="-2.54" width="0.1524" layer="91"/>
-<label x="238.76" y="-2.54" size="1.778" layer="95"/>
-</segment>
-</net>
-<net name="GPIO3" class="0">
-<segment>
-<pinref part="U2" gate="A" pin="PA6/PGMNOE"/>
-<wire x1="393.7" y1="71.12" x2="408.94" y2="71.12" width="0.1524" layer="91"/>
-<label x="401.32" y="71.12" size="1.778" layer="95"/>
-</segment>
-<segment>
-<pinref part="U$2" gate="G$1" pin="PIO3_14/DP09A"/>
-<wire x1="233.68" y1="0" x2="246.38" y2="0" width="0.1524" layer="91"/>
-<label x="238.76" y="0" size="1.778" layer="95"/>
-</segment>
-</net>
-<net name="GPIO4" class="0">
-<segment>
-<pinref part="U2" gate="A" pin="PA8/XOUT32/PGMM0"/>
-<wire x1="393.7" y1="66.04" x2="408.94" y2="66.04" width="0.1524" layer="91"/>
-<label x="401.32" y="66.04" size="1.778" layer="95"/>
-</segment>
-<segment>
-<pinref part="U$2" gate="G$1" pin="PIO3_13/DP08B"/>
-<wire x1="233.68" y1="2.54" x2="246.38" y2="2.54" width="0.1524" layer="91"/>
-<label x="238.76" y="2.54" size="1.778" layer="95"/>
-</segment>
-</net>
-<net name="GPIO5" class="0">
-<segment>
-<pinref part="U2" gate="A" pin="PA15/PGMD3"/>
-<wire x1="393.7" y1="48.26" x2="411.48" y2="48.26" width="0.1524" layer="91"/>
-<label x="403.86" y="48.26" size="1.778" layer="95"/>
-</segment>
-<segment>
-<pinref part="U$2" gate="G$1" pin="PIO3_11/DP04B"/>
-<wire x1="233.68" y1="7.62" x2="246.38" y2="7.62" width="0.1524" layer="91"/>
-<label x="238.76" y="7.62" size="1.778" layer="95"/>
-</segment>
-</net>
-<net name="GPIO6" class="0">
-<segment>
-<pinref part="U2" gate="A" pin="PA16/PGMD4"/>
-<wire x1="393.7" y1="45.72" x2="411.48" y2="45.72" width="0.1524" layer="91"/>
-<label x="403.86" y="45.72" size="1.778" layer="95"/>
-</segment>
-<segment>
-<pinref part="U$2" gate="G$1" pin="PIO3_12/DP07A"/>
-<wire x1="233.68" y1="5.08" x2="246.38" y2="5.08" width="0.1524" layer="91"/>
-<label x="238.76" y="5.08" size="1.778" layer="95"/>
-</segment>
-</net>

Commit message: new GND layer
Changed lines of the file:
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@@
 <pinref part="U$2" gate="G$1" pin="PIO2_05"/>
 <wire x1="233.68" y1="78.74" x2="256.54" y2="78.74" width="0.1524" layer="91"/>
+<label x="248.92" y="78.74" size="1.778" layer="95"/>
 </segment>
 </net>
@@
 <pinref part="U$2" gate="G$1" pin="PIO2_06"/>
 <wire x1="233.68" y1="76.2" x2="256.54" y2="76.2" width="0.1524" layer="91"/>
+<label x="248.92" y="76.2" size="1.778" layer="95"/>
 </segment>
 </net>
