File: board/tinz.sch (EAGLE design)
At the start: 110 parts, among them U2 ATSAM3S4AA-AU

Commit message: Fixed some bugs.
Connections:
- net MISO: now also U$2.PIOS_01/SPI_SI; no longer U$2.PIOS_02/SPI_SO
- net MOSI: now also U$2.PIOS_02/SPI_SO; no longer U$2.PIOS_01/SPI_SI
Changed lines of the file:
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@@
 <?xml version="1.0" encoding="utf-8"?>
 <!DOCTYPE eagle SYSTEM "eagle.dtd">
-<eagle version="7.4.0">
+<eagle version="7.5.0">
 <drawing>
 <settings>
@@
 <net name="MOSI" class="0">
 <segment>
+<label x="122.682" y="128.778" size="1.778" layer="95"/>
+<pinref part="U$1" gate="G$1" pin="ACBUS1"/>
+<wire x1="121.92" y1="129.54" x2="101.6" y2="129.54" width="0.1524" layer="91"/>
+</segment>
+<segment>
+<pinref part="U$3" gate="G$1" pin="DQ0"/>
+<wire x1="58.42" y1="-7.62" x2="10.16" y2="-7.62" width="0.1524" layer="91"/>
+<label x="3.302" y="-8.382" size="1.778" layer="95"/>
+</segment>
+<segment>
+<pinref part="U$2" gate="G$1" pin="PIOS_02/SPI_SO"/>
+<wire x1="182.88" y1="127" x2="180.34" y2="127" width="0.1524" layer="91"/>
+<label x="173.736" y="126.238" size="1.778" layer="95"/>
+</segment>
+</net>
+<net name="MISO" class="0">
+<segment>
+<label x="122.682" y="126.238" size="1.778" layer="95"/>
+<pinref part="U$1" gate="G$1" pin="ACBUS2"/>
+<wire x1="121.92" y1="127" x2="101.6" y2="127" width="0.1524" layer="91"/>
+</segment>
+<segment>
+<pinref part="U$3" gate="G$1" pin="DQ1"/>
+<wire x1="91.44" y1="-12.7" x2="93.98" y2="-12.7" width="0.1524" layer="91"/>
+<label x="93.98" y="-12.7" size="1.778" layer="95"/>
+</segment>
+<segment>
 <pinref part="U$2" gate="G$1" pin="PIOS_01/SPI_SI"/>
 <wire x1="182.88" y1="129.54" x2="180.34" y2="129.54" width="0.1524" layer="91"/>
 <label x="173.736" y="128.778" size="1.778" layer="95"/>
 </segment>
-<segment>
-<label x="122.682" y="128.778" size="1.778" layer="95"/>
-<pinref part="U$1" gate="G$1" pin="ACBUS1"/>
-<wire x1="121.92" y1="129.54" x2="101.6" y2="129.54" width="0.1524" layer="91"/>
-</segment>
-<segment>
-<pinref part="U$3" gate="G$1" pin="DQ0"/>
-<wire x1="58.42" y1="-7.62" x2="10.16" y2="-7.62" width="0.1524" layer="91"/>
-<label x="3.302" y="-8.382" size="1.778" layer="95"/>
-</segment>
-</net>
-<net name="MISO" class="0">
-<segment>
-<pinref part="U$2" gate="G$1" pin="PIOS_02/SPI_SO"/>
-<wire x1="182.88" y1="127" x2="180.34" y2="127" width="0.1524" layer="91"/>
-<label x="173.99" y="126.238" size="1.778" layer="95"/>
-</segment>
-<segment>
-<label x="122.682" y="126.238" size="1.778" layer="95"/>
-<pinref part="U$1" gate="G$1" pin="ACBUS2"/>
-<wire x1="121.92" y1="127" x2="101.6" y2="127" width="0.1524" layer="91"/>
-</segment>
-<segment>
-<pinref part="U$3" gate="G$1" pin="DQ1"/>
-<wire x1="91.44" y1="-12.7" x2="93.98" y2="-12.7" width="0.1524" layer="91"/>
-<label x="93.98" y="-12.7" size="1.778" layer="95"/>
-</segment>
-</net>
+</net>

Commit message: Added an inverter chip.
Parts:
- added IC1: 74LVC1G14DCK, 74xx-little-us:74LVC1G14DCK
Connections:
- new net N$8: IC1A.O, U2.ERASE/PB12
- net DTRN: now also IC1A.I; no longer U2.ERASE/PB12
Changed lines of the file:
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@@
 <?xml version="1.0" encoding="utf-8"?>
 <!DOCTYPE eagle SYSTEM "eagle.dtd">
-<eagle version="7.5.0">
+<eagle version="7.4.0">
 <drawing>
 <settings>
@@
 <part name="SUPPLY20" library="supply2" deviceset="GND" device=""/>
 <part name="U$8" library="ecx32" deviceset="ECO32" device=""/>
+<part name="IC1" library="74xx-little-us" deviceset="74*1G14" device="DCK" technology="LVC"/>
 </parts>
 <sheets>
@@
 <attribute name="VALUE" x="472.44" y="91.44" size="1.778" layer="96" rot="R180"/>
 </instance>
+<instance part="IC1" gate="A" x="424.18" y="27.94" rot="R180"/>
 </instances>
 <busses>
@@
 </segment>
 <segment>
-<pinref part="U2" gate="A" pin="ERASE/PB12"/>
-<wire x1="393.7" y1="27.94" x2="408.94" y2="27.94" width="0.1524" layer="91"/>
-<label x="401.32" y="27.94" size="1.778" layer="95"/>
+<pinref part="IC1" gate="A" pin="I"/>
+<wire x1="434.34" y1="27.94" x2="441.96" y2="27.94" width="0.1524" layer="91"/>
+<label x="436.88" y="27.94" size="1.778" layer="95"/>
 </segment>
 </net>
@@
 </segment>
 </net>
+<net name="N$8" class="0">
+<segment>
+<pinref part="IC1" gate="A" pin="O"/>
+<pinref part="U2" gate="A" pin="ERASE/PB12"/>
+<wire x1="414.02" y1="27.94" x2="393.7" y2="27.94" width="0.1524" layer="91"/>
+</segment>
+</net>

Commit message: Fixed LED size issue.
Parts:
- LED1, LED2, LED3, LED4, LED5, LED6, LED7, LED8: device led:LEDSMT1206 -> led:LEDSML0603
Changed lines of the file:
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@@
 <grid distance="0.1" unitdist="inch" unit="inch" style="lines" multiple="1" display="no" altdistance="0.01" altunitdist="inch" altunit="inch"/>
 <layers>
-<layer number="1" name="Top" color="4" fill="1" visible="no" active="no"/>
-<layer number="16" name="Bottom" color="1" fill="1" visible="no" active="no"/>
-<layer number="17" name="Pads" color="2" fill="1" visible="no" active="no"/>
-<layer number="18" name="Vias" color="2" fill="1" visible="no" active="no"/>
-<layer number="19" name="Unrouted" color="6" fill="1" visible="no" active="no"/>
-<layer number="20" name="Dimension" color="15" fill="1" visible="no" active="no"/>
-<layer number="21" name="tPlace" color="7" fill="1" visible="no" active="no"/>
-<layer number="22" name="bPlace" color="7" fill="1" visible="no" active="no"/>
-<layer number="23" name="tOrigins" color="15" fill="1" visible="no" active="no"/>
-<layer number="24" name="bOrigins" color="15" fill="1" visible="no" active="no"/>
-<layer number="25" name="tNames" color="7" fill="1" visible="no" active="no"/>
-<layer number="26" name="bNames" color="7" fill="1" visible="no" active="no"/>
-<layer number="27" name="tValues" color="7" fill="1" visible="no" active="no"/>
-<layer number="28" name="bValues" color="7" fill="1" visible="no" active="no"/>
+<layer number="1" name="Top" color="4" fill="1" visible="yes" active="no"/>
+<layer number="16" name="Bottom" color="1" fill="1" visible="yes" active="no"/>
+<layer number="17" name="Pads" color="2" fill="1" visible="yes" active="no"/>
+<layer number="18" name="Vias" color="2" fill="1" visible="yes" active="no"/>
+<layer number="19" name="Unrouted" color="6" fill="1" visible="yes" active="no"/>
+<layer number="20" name="Dimension" color="15" fill="1" visible="yes" active="no"/>
+<layer number="21" name="tPlace" color="7" fill="1" visible="yes" active="no"/>
+<layer number="22" name="bPlace" color="7" fill="1" visible="yes" active="no"/>
+<layer number="23" name="tOrigins" color="15" fill="1" visible="yes" active="no"/>
+<layer number="24" name="bOrigins" color="15" fill="1" visible="yes" active="no"/>
+<layer number="25" name="tNames" color="7" fill="1" visible="yes" active="no"/>
+<layer number="26" name="bNames" color="7" fill="1" visible="yes" active="no"/>
+<layer number="27" name="tValues" color="7" fill="1" visible="yes" active="no"/>
+<layer number="28" name="bValues" color="7" fill="1" visible="yes" active="no"/>
 <layer number="29" name="tStop" color="7" fill="3" visible="no" active="no"/>
 <layer number="30" name="bStop" color="7" fill="6" visible="no" active="no"/>
@@
 <layer number="35" name="tGlue" color="7" fill="4" visible="no" active="no"/>
 <layer number="36" name="bGlue" color="7" fill="5" visible="no" active="no"/>
-<layer number="37" name="tTest" color="7" fill="1" visible="no" active="no"/>
-<layer number="38" name="bTest" color="7" fill="1" visible="no" active="no"/>
+<layer number="37" name="tTest" color="7" fill="1" visible="yes" active="no"/>
+<layer number="38" name="bTest" color="7" fill="1" visible="yes" active="no"/>
 <layer number="39" name="tKeepout" color="4" fill="11" visible="no" active="no"/>
 <layer number="40" name="bKeepout" color="1" fill="11" visible="no" active="no"/>
@@
 <layer number="44" name="Drills" color="7" fill="1" visible="no" active="no"/>
 <layer number="45" name="Holes" color="7" fill="1" visible="no" active="no"/>
-<layer number="46" name="Milling" color="3" fill="1" visible="no" active="no"/>
-<layer number="47" name="Measures" color="7" fill="1" visible="no" active="no"/>
-<layer number="48" name="Document" color="7" fill="1" visible="no" active="no"/>
-<layer number="49" name="Reference" color="7" fill="1" visible="no" active="no"/>
-<layer number="50" name="dxf" color="7" fill="1" visible="no" active="no"/>
-<layer number="51" name="tDocu" color="7" fill="1" visible="no" active="no"/>
-<layer number="52" name="bDocu" color="7" fill="1" visible="no" active="no"/>
-<layer number="53" name="tGND_GNDA" color="7" fill="9" visible="no" active="no"/>
-<layer number="54" name="bGND_GNDA" color="1" fill="9" visible="no" active="no"/>
-<layer number="56" name="wert" color="7" fill="1" visible="no" active="no"/>
-<layer number="57" name="tCAD" color="7" fill="1" visible="no" active="no"/>
-<layer number="59" name="tCarbon" color="7" fill="1" visible="no" active="no"/>
-<layer number="60" name="bCarbon" color="7" fill="1" visible="no" active="no"/>
+<layer number="46" name="Milling" color="3" fill="1" visible="yes" active="no"/>
+<layer number="47" name="Measures" color="7" fill="1" visible="yes" active="no"/>
+<layer number="48" name="Document" color="7" fill="1" visible="yes" active="no"/>
+<layer number="49" name="Reference" color="7" fill="1" visible="yes" active="no"/>
+<layer number="50" name="dxf" color="7" fill="1" visible="yes" active="no"/>
+<layer number="51" name="tDocu" color="7" fill="1" visible="yes" active="no"/>
+<layer number="52" name="bDocu" color="7" fill="1" visible="yes" active="no"/>
+<layer number="53" name="tGND_GNDA" color="7" fill="9" visible="yes" active="no"/>
+<layer number="54" name="bGND_GNDA" color="1" fill="9" visible="yes" active="no"/>
+<layer number="56" name="wert" color="7" fill="1" visible="yes" active="no"/>
+<layer number="57" name="tCAD" color="7" fill="1" visible="yes" active="no"/>
+<layer number="59" name="tCarbon" color="7" fill="1" visible="yes" active="no"/>
+<layer number="60" name="bCarbon" color="7" fill="1" visible="yes" active="no"/>
 <layer number="90" name="Modules" color="5" fill="1" visible="yes" active="yes"/>
 <layer number="91" name="Nets" color="2" fill="1" visible="yes" active="yes"/>
@@
 <part name="SUPPLY14" library="supply2" deviceset="GND" device=""/>
 <part name="R37" library="resistor" deviceset="R-US_" device="R0603" value="100"/>
-<part name="LED1" library="led" deviceset="LED" device="SMT1206" value="Green"/>
-<part name="LED2" library="led" deviceset="LED" device="SMT1206" value="Green"/>
-<part name="LED3" library="led" deviceset="LED" device="SMT1206" value="Green"/>
-<part name="LED4" library="led" deviceset="LED" device="SMT1206" value="Green"/>
+<part name="LED1" library="led" deviceset="LED" device="SML0603" value="Green"/>
+<part name="LED2" library="led" deviceset="LED" device="SML0603" value="Green"/>
+<part name="LED3" library="led" deviceset="LED" device="SML0603" value="Green"/>
+<part name="LED4" library="led" deviceset="LED" device="SML0603" value="Green"/>
 <part name="R38" library="resistor" deviceset="R-US_" device="R0603" value="100"/>
 <part name="R39" library="resistor" deviceset="R-US_" device="R0603" value="100"/>
 <part name="R40" library="resistor" deviceset="R-US_" device="R0603" value="100"/>
 <part name="SUPPLY21" library="supply2" deviceset="GND" device=""/>
-<part name="LED5" library="led" deviceset="LED" device="SMT1206" value="Amber"/>
-<part name="LED6" library="led" deviceset="LED" device="SMT1206" value="Amber"/>
+<part name="LED5" library="led" deviceset="LED" device="SML0603" value="Amber"/>
+<part name="LED6" library="led" deviceset="LED" device="SML0603" value="Amber"/>
 <part name="R41" library="resistor" deviceset="R-US_" device="R0603" value="100"/>
 <part name="R42" library="resistor" deviceset="R-US_" device="R0603" value="100"/>
 <part name="SUPPLY22" library="supply2" deviceset="GND" device=""/>
-<part name="LED7" library="led" deviceset="LED" device="SMT1206" value="Red"/>
-<part name="LED8" library="led" deviceset="LED" device="SMT1206" value="Red"/>
+<part name="LED7" library="led" deviceset="LED" device="SML0603" value="Red"/>
+<part name="LED8" library="led" deviceset="LED" device="SML0603" value="Red"/>
 <part name="R43" library="resistor" deviceset="R-US_" device="R0603" value="25"/>
 <part name="R44" library="resistor" deviceset="R-US_" device="R0603" value="100"/>
