File: board/tinz.brd (EAGLE design)
At the start: 101.3 x 80 mm, 111 parts, among them U2 ATSAM3S4AA-AU

Commit message: Routed USB stuff.
Routing:
- net D_N: track 0.00 -> 32.3 mm, vias 0 -> 1
- net D_P: track 0.00 -> 32.3 mm, vias 0 -> 2
- net GND: track 169.9 -> 172.1 mm
Changed lines of the file:
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@@
 <contactref element="U$6" pad="P$18"/>
 <contactref element="U$6" pad="P$19"/>
+<wire x1="10.635" y1="59.9" x2="9.575" y2="59.9" width="0.3048" layer="1"/>
+<wire x1="9.575" y1="59.9" x2="9.525" y2="59.95" width="0.3048" layer="1"/>
+<wire x1="10.635" y1="54.4" x2="9.575" y2="54.4" width="0.3048" layer="1"/>
+<wire x1="9.575" y1="54.4" x2="9.525" y2="54.35" width="0.3048" layer="1"/>
 <wire x1="67.945" y1="77.685" x2="69.85" y2="75.985" width="0" layer="19" extent="1-1"/>
 <wire x1="66.04" y1="75.985" x2="67.945" y2="77.685" width="0" layer="19" extent="1-1"/>
@@
 <wire x1="41.91" y1="67.31" x2="50.8" y2="75.35" width="0" layer="19" extent="1-1"/>
 <wire x1="6.985" y1="30.48" x2="7.86" y2="30.48" width="0" layer="19" extent="1-1"/>
-<wire x1="10.635" y1="59.9" x2="9.525" y2="59.95" width="0" layer="19" extent="1-1"/>
-<wire x1="10.635" y1="54.4" x2="9.525" y2="54.35" width="0" layer="19" extent="1-1"/>
 <wire x1="33.715" y1="57.345" x2="33.715" y2="59.345" width="0" layer="19" extent="1-1"/>
 <wire x1="33.715" y1="54.845" x2="33.715" y2="57.345" width="0" layer="19" extent="1-1"/>
@@
 <contactref element="U$6" pad="A7"/>
 <contactref element="U$1" pad="7"/>
-<wire x1="10.635" y1="56.9" x2="33.715" y2="56.345" width="0" layer="19" extent="1-1"/>
-<wire x1="9.525" y1="57.55" x2="10.635" y2="56.9" width="0" layer="19" extent="1-1"/>
+<wire x1="10.635" y1="56.9" x2="12.315" y2="56.9" width="0.2032" layer="1"/>
+<wire x1="12.315" y1="56.9" x2="12.7" y2="56.515" width="0.2032" layer="1"/>
+<via x="12.7" y="56.515" extent="1-16" drill="0.4" shape="octagon"/>
+<wire x1="9.525" y1="57.55" x2="11.665" y2="57.55" width="0.2032" layer="16"/>
+<wire x1="11.665" y1="57.55" x2="12.7" y2="56.515" width="0.2032" layer="16"/>
+<wire x1="12.7" y1="56.515" x2="15.1067125" y2="59.20908125" width="0.2032" layer="1"/>
+<wire x1="15.1067125" y1="59.20908125" x2="17.69583125" y2="61.7982" width="0.2032" layer="1"/>
+<wire x1="17.69583125" y1="61.7982" x2="23.57916875" y2="61.7982" width="0.2032" layer="1"/>
+<wire x1="23.57916875" y1="61.7982" x2="26.8732" y2="58.50416875" width="0.2032" layer="1"/>
+<wire x1="26.8732" y1="58.50416875" x2="26.8732" y2="57.23416875" width="0.2032" layer="1"/>
+<wire x1="26.8732" y1="57.23416875" x2="28.02416875" y2="56.0832" width="0.2032" layer="1"/>
+<wire x1="28.02416875" y1="56.0832" x2="31.115" y2="56.0832" width="0.2032" layer="1"/>
+<wire x1="31.115" y1="56.0832" x2="31.3768" y2="56.345" width="0.2032" layer="1"/>
+<wire x1="31.3768" y1="56.345" x2="33.715" y2="56.345" width="0.2032" layer="1"/>
 </signal>
 <signal name="D_P" class="2">
@@
 <contactref element="U$6" pad="A6"/>
 <contactref element="U$1" pad="8"/>
-<wire x1="10.635" y1="57.4" x2="33.715" y2="55.845" width="0" layer="19" extent="1-1"/>
-<wire x1="9.525" y1="56.75" x2="10.635" y2="57.4" width="0" layer="19" extent="1-1"/>
+<wire x1="33.68" y1="55.88" x2="33.715" y2="55.845" width="0.2032" layer="1"/>
+<wire x1="10.635" y1="57.4" x2="10.175" y2="57.4" width="0.2032" layer="1"/>
+<wire x1="10.175" y1="57.4" x2="9.525" y2="56.75" width="0.2032" layer="1"/>
+<wire x1="10.635" y1="57.4" x2="12.315" y2="57.4" width="0.2032" layer="1"/>
+<wire x1="12.315" y1="57.4" x2="12.7" y2="57.785" width="0.2032" layer="1"/>
+<via x="12.7" y="57.785" extent="1-16" drill="0.4" shape="octagon"/>
+<wire x1="12.7" y1="57.785" x2="12.7" y2="57.15" width="0.2032" layer="16"/>
+<wire x1="12.7" y1="57.15" x2="13.97" y2="55.88" width="0.2032" layer="16"/>
+<via x="13.97" y="55.88" extent="1-16" drill="0.4" shape="octagon"/>
+<wire x1="13.97" y1="55.88" x2="14.8082" y2="56.515" width="0.2032" layer="1"/>
+<wire x1="14.8082" y1="56.515" x2="14.8082" y2="58.33583125" width="0.2032" layer="1"/>
+<wire x1="14.8082" y1="58.33583125" x2="17.86416875" y2="61.3918" width="0.2032" layer="1"/>
+<wire x1="17.86416875" y1="61.3918" x2="23.41083125" y2="61.3918" width="0.2032" layer="1"/>
+<wire x1="23.41083125" y1="61.3918" x2="26.4668" y2="58.33583125" width="0.2032" layer="1"/>
+<wire x1="26.4668" y1="58.33583125" x2="26.4668" y2="57.06583125" width="0.2032" layer="1"/>
+<wire x1="26.4668" y1="57.06583125" x2="27.85583125" y2="55.6768" width="0.2032" layer="1"/>
+<wire x1="27.85583125" y1="55.6768" x2="31.115" y2="55.6768" width="0.2032" layer="1"/>
+<wire x1="31.115" y1="55.6768" x2="31.2832" y2="55.845" width="0.2032" layer="1"/>
+<wire x1="31.2832" y1="55.845" x2="33.715" y2="55.845" width="0.2032" layer="1"/>
 </signal>
 </signals>

Commit message: Untwisted most of the wires between the MCU and GPIO.
Parts:
- moved C26 1.42 mm to (56.5, 15.9), turned to 90 degrees
- moved C29 1.27 mm to (59.7, 19.7)
- moved C33 1.27 mm to (56.5, 19.7)
Connections:
- net GPIO0: now also U$2.26; no longer U$2.12
- net GPIO1: now also U$2.25; no longer U$2.19
- net GPIO2: now also U$2.24; no longer U$2.20
- net GPIO3: now also U$2.23; no longer U$2.21
- net GPIO5: now also U$2.12; no longer U$2.23
- net GPIO6: now also U$2.19; no longer U$2.24
- net GPIO7: now also U$2.21; no longer U$2.25
- net GPIO8: now also U$2.20; no longer U$2.26
- net M_MISO: now also U$2.47; no longer U$2.48
- net M_MOSI: now also U$2.48; no longer U$2.47
- net TWCK0: now also U$2.2; no longer U$2.3
- net TWD0: now also U$2.3; no longer U$2.2
Routing:
- net UTXD0: track 0.00 -> 62.9 mm, vias 0 -> 2
- net URXD0: track 0.00 -> 59.4 mm, vias 0 -> 2

Commit message: Just some PCB stuff.
Parts:
- moved C11 4.37 mm to (59.1, 29.6), turned to 0 degrees
- moved C12 2.84 mm to (59.1, 31.8), turned to 0 degrees
- moved C17 1.27 mm to (71.1, 76.8)
- moved C20 0.64 mm to (68.6, 76.8), turned to 270 degrees
Routing:
- net GND: track 172.1 -> 211.0 mm, vias 15 -> 33
- net N$9: track 0.00 -> 5.74 mm
- net +1.2V: track 128.0 -> 130.4 mm
- net +3.3V: track 25.1 -> 23.8 mm

Commit message: Ran the TWI and UART traces
Parts:
- moved R47 2.54 mm to (80.2, 42.6)
- moved R46 2.54 mm to (77.8, 42.6)
Connections:
- net TWCK0: now also U$2.39; no longer U$2.2
- net TWD0: now also U$2.38; no longer U$2.3
Routing:
- net TWCK0: track 6.09 -> 47.9 mm
- net TWD0: track 5.81 -> 43.4 mm
- net UTXD1: track 0.00 -> 32.8 mm, vias 0 -> 2
- net FT_EEDATA: track 0.00 -> 31.2 mm
- net URXD1: track 1.83 -> 32.9 mm, vias 1 -> 2
- net FT_EECLK: track 0.00 -> 27.2 mm
- net FT_EECS: track 0.00 -> 26.1 mm
- net N$10: track 0.00 -> 9.50 mm
- net SPI_NPCS0: track 0.00 -> 4.87 mm, vias 0 -> 1
- net GND: track 211.0 -> 212.3 mm

Commit message: Routed SPI
Routing:
- net M_SPCK: track 0.00 -> 71.3 mm, vias 0 -> 4
- net M_MOSI: track 0.00 -> 70.2 mm, vias 0 -> 2
- net M_MISO: track 0.00 -> 68.4 mm, vias 0 -> 2
- net SPI_NPCS0: track 4.87 -> 72.2 mm, vias 1 -> 2
- net VCC1_8FT: track 9.70 -> 39.1 mm
- net +3.3V: track 23.6 -> 17.8 mm
- net +1.2V: track 130.4 -> 133.2 mm
