File: board/tinz.brd (EAGLE design)
At the start: 101.3 x 80 mm, 111 parts, among them U2 ATSAM3S4AA-AU

Commit message: Some more wires added.
Parts:
- removed R14: 0, resistor:R0603
- moved C37 4.07 mm to (27.9, 50.8), turned to 0 degrees
- moved R28 1.27 mm to (26.7, 53.3)
Connections:
- removed net N$11: R14.1, U$2.66
- net CRESET_B: now also U$2.66; no longer R14.2
- net GPIO0: now also U2.35; no longer U2.36
- net GPIO1: now also U2.36; no longer U2.35
Routing:
- net DTRN: track 0.00 -> 53.9 mm, vias 0 -> 2
- net +3.3V: track 17.8 -> 42.5 mm
- net VDDOUT: track 12.0 -> 29.8 mm
- net VBUS_5V: track 43.1 -> 59.9 mm
- net GND: track 212.3 -> 222.0 mm, vias 33 -> 36
- net CRESET_B: track 13.1 -> 18.0 mm, vias 0 -> 2
- net N$11: track 3.67 -> 0.00 mm
- net N$19: track 5.13 -> 6.40 mm

Commit message: IDK
Routing:
- net GPIO0: track 0.00 -> 33.7 mm
- net GPIO1: track 0.00 -> 31.6 mm
Changed lines of the file:
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@@
 <wire x1="72.6694" y1="26.9494" x2="72.39" y2="26.67" width="0.3048" layer="1"/>
 <wire x1="74.93" y1="38.315" x2="76.8604" y2="33.4518" width="0" layer="19" extent="1-1"/>
+<wire x1="37.465" y1="38.735" x2="42.35" y2="37.42" width="0" layer="19" extent="1-1"/>
+<wire x1="33.715" y1="55.345" x2="37.465" y2="51.435" width="0" layer="19" extent="1-1"/>
 <wire x1="3.81" y1="44.03" x2="4.445" y2="44.665" width="0" layer="19" extent="1-1"/>
 <wire x1="3.175" y1="44.03" x2="3.81" y2="44.03" width="0" layer="19" extent="1-1"/>
 <wire x1="41.275" y1="17.145" x2="36.83" y2="17.78" width="0" layer="19" extent="1-1"/>
 <wire x1="27.35" y1="27.42" x2="24.13" y2="31.33" width="0" layer="19" extent="1-1"/>
-<wire x1="37.465" y1="38.735" x2="42.35" y2="37.42" width="0" layer="19" extent="1-1"/>
 </signal>
 <signal name="FT_EECLK">
@@
 <contactref element="U$2" pad="26"/>
 <contactref element="U2" pad="35"/>
-<wire x1="48.85" y1="30.42" x2="75.8444" y2="33.4518" width="0" layer="19" extent="1-1"/>
+<wire x1="75.8444" y1="33.4518" x2="75.8444" y2="34.6456" width="0.3048" layer="1"/>
+<wire x1="75.8444" y1="34.6456" x2="75.565" y2="34.925" width="0.3048" layer="1"/>
+<wire x1="75.565" y1="34.925" x2="74.93" y2="34.925" width="0.3048" layer="1"/>
+<wire x1="74.93" y1="34.925" x2="74.295" y2="34.29" width="0.3048" layer="1"/>
+<wire x1="74.295" y1="34.29" x2="66.675" y2="34.29" width="0.3048" layer="1"/>
+<wire x1="66.675" y1="34.29" x2="63.5" y2="31.115" width="0.3048" layer="1"/>
+<wire x1="63.5" y1="31.115" x2="63.5" y2="28.575" width="0.3048" layer="1"/>
+<wire x1="63.5" y1="28.575" x2="62.865" y2="27.94" width="0.3048" layer="1"/>
+<wire x1="62.865" y1="27.94" x2="57.785" y2="27.94" width="0.3048" layer="1"/>
+<wire x1="57.785" y1="27.94" x2="55.305" y2="30.42" width="0.3048" layer="1"/>
+<wire x1="55.305" y1="30.42" x2="48.85" y2="30.42" width="0.3048" layer="1"/>
 </signal>
 <signal name="GPIO1">
 <contactref element="U$2" pad="25"/>
 <contactref element="U2" pad="36"/>
-<wire x1="48.85" y1="29.92" x2="75.3618" y2="33.4518" width="0" layer="19" extent="1-1"/>
+<wire x1="75.3618" y1="33.4518" x2="67.1068" y2="33.4518" width="0.3048" layer="1"/>
+<wire x1="67.1068" y1="33.4518" x2="64.135" y2="30.48" width="0.3048" layer="1"/>
+<wire x1="64.135" y1="30.48" x2="64.135" y2="27.94" width="0.3048" layer="1"/>
+<wire x1="64.135" y1="27.94" x2="63.5" y2="27.305" width="0.3048" layer="1"/>
+<wire x1="63.5" y1="27.305" x2="57.15" y2="27.305" width="0.3048" layer="1"/>
+<wire x1="57.15" y1="27.305" x2="54.535" y2="29.92" width="0.3048" layer="1"/>
+<wire x1="54.535" y1="29.92" x2="48.85" y2="29.92" width="0.3048" layer="1"/>
 </signal>
 <signal name="GPIO2">

Commit message: Added the ecx crystal oscillator.
Parts:
- removed Q1: (no value), crystal:HC49UP
- added U$8: ECO32, ecx32:4-SMD
- moved C53 11.1 mm to (72.4, 14.6)
- moved C54 11.1 mm to (66.0, 14.6)
- moved C32 1.27 mm to (52.1, 34.3)
- moved C31 0.63 mm to (54.6, 34.3)
- moved C40 0.30 mm to (53.3, 52.4)
- moved C39 0.15 mm to (53.3, 54.5)
Connections:
- removed net GPIO2: U$2.24, U2.32
- removed net GPIO3: U$2.23, U2.26
- removed net GPIO4: U$2.22, U2.23
- removed net GPIO5: U$2.12, U2.15
- removed net GPIO6: U$2.19, U2.14
- removed net GPIO7: U$2.21, U2.43
- removed net GPIO8: U$2.20, U2.44
- net GND: now also U$8.2, U$8.4
- net XIN: now also U$8.1; no longer Q1.2
- net XOUT: now also U$8.3; no longer Q1.1
Routing:
- net GND: track 222.0 -> 240.3 mm, vias 36 -> 38
- net XOUT: track 0.00 -> 17.4 mm
- net XIN: track 0.00 -> 15.0 mm
- net +3.3V: track 42.5 -> 47.3 mm, vias 2 -> 4
- net N$9: track 5.74 -> 6.84 mm

Commit message: new GND layer
Parts:
- moved C28 0.81 mm to (53.7, 19.7), turned to 90 degrees
- moved C29 0.63 mm to (59.1, 19.7), turned to 90 degrees
- moved C22 0.63 mm to (60.3, 76.8)
- turned C26 to 270 degrees
- turned C30 to 270 degrees
- turned C33 to 90 degrees
Routing:
- net GND: track 240.3 -> 80.2 mm, vias 38 -> 2
- net +3.3V: track 47.3 -> 104.5 mm
- added copper zone on layer 1, net GND
- removed copper zone on layer 1, net +3.3V

Commit message: Got most of it done!
Parts:
- moved C14 9.44 mm to (10.2, 50.8)
- moved U$6 1.70 mm to (7.82, 57.1)
Routing:
- net +3.3V: track 104.5 -> 678.7 mm, vias 4 -> 10
- net GND: track 80.2 -> 87.2 mm, vias 2 -> 17
- net D_P: track 32.3 -> 34.0 mm
- net D_N: track 32.3 -> 34.0 mm
- net VCC1_8FT: track 39.1 -> 39.7 mm
- net SS: track 33.2 -> 33.8 mm
- net MISO: track 25.5 -> 26.1 mm
- net VBUS_5V: track 60.1 -> 60.6 mm

Commit message: I think the board is finished.
Parts:
- moved C13 44.7 mm to (48.9, 48.3), turned to 0 degrees
- moved C14 38.7 mm to (48.9, 50.2), turned to 0 degrees
- moved C15 34.9 mm to (24.1, 15.2), turned to 0 degrees
- moved C16 14.3 mm to (17.1, 38.1)
Routing:
- net +3.3V: track 678.7 -> 690.7 mm
- net GND: track 87.2 -> 86.0 mm
