File: board/tinz.brd (EAGLE design)
At the start: 101.3 x 80 mm, 110 parts, among them U2 ATSAM3S4AA-AU

Commit message: Changed shape of vias. Fixed some issues.
Parts:
- moved C45 0.64 mm to (67.9, 27.3)
- moved C8 0.63 mm to (39.4, 12.7)
Routing:
- net DTRN: track 53.9 -> 54.4 mm
Changed lines of the file:
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@@
 <layer number="27" name="tValues" color="7" fill="1" visible="no" active="yes"/>
 <layer number="28" name="bValues" color="7" fill="1" visible="no" active="yes"/>
-<layer number="29" name="tStop" color="7" fill="3" visible="no" active="yes"/>
-<layer number="30" name="bStop" color="7" fill="6" visible="no" active="yes"/>
+<layer number="29" name="tStop" color="7" fill="3" visible="yes" active="yes"/>
+<layer number="30" name="bStop" color="7" fill="6" visible="yes" active="yes"/>
 <layer number="31" name="tCream" color="7" fill="4" visible="no" active="yes"/>
 <layer number="32" name="bCream" color="7" fill="5" visible="no" active="yes"/>
@@
 <attribute name="VALUE" x="87.63" y="29.845" size="1.27" layer="27"/>
 </element>
-<element name="C45" library="resistor" package="C0603" value="10uF" x="67.945" y="27.94" smashed="yes">
-<attribute name="NAME" x="62.865" y="27.305" size="1.27" layer="25"/>
-<attribute name="VALUE" x="67.31" y="26.035" size="1.27" layer="27"/>
+<element name="C45" library="resistor" package="C0603" value="10uF" x="67.945" y="27.305" smashed="yes">
+<attribute name="NAME" x="62.865" y="26.67" size="1.27" layer="25"/>
+<attribute name="VALUE" x="67.31" y="25.4" size="1.27" layer="27"/>
 </element>
 <element name="C46" library="resistor" package="C0603" value="10uF" x="74.93" y="37.465" smashed="yes" rot="R270">
@@
 <attribute name="VALUE" x="36.195" y="8.255" size="1.27" layer="27" rot="R90"/>
 </element>
-<element name="C8" library="resistor" package="C0603" value="0.1uF" x="38.735" y="12.7" smashed="yes">
-<attribute name="NAME" x="37.465" y="13.335" size="1.27" layer="25"/>
-<attribute name="VALUE" x="38.1" y="10.795" size="1.27" layer="27"/>
+<element name="C8" library="resistor" package="C0603" value="0.1uF" x="39.37" y="12.7" smashed="yes">
+<attribute name="NAME" x="38.1" y="13.335" size="1.27" layer="25"/>
+<attribute name="VALUE" x="38.735" y="10.795" size="1.27" layer="27"/>
 </element>
 <element name="C9" library="resistor" package="C0603" value="0.1uF" x="24.13" y="26.67" smashed="yes" rot="R90">
@@
 <via x="37.465" y="6.35" extent="1-16" drill="0.5" shape="octagon"/>
 <wire x1="37.465" y1="8.04" x2="37.465" y2="6.35" width="0.3048" layer="1"/>
-<via x="36.576" y="13.081" extent="1-16" drill="0.6" shape="octagon"/>
-<wire x1="37.885" y1="12.7" x2="36.957" y2="12.7" width="0.3048" layer="1"/>
-<wire x1="36.957" y1="12.7" x2="36.576" y2="13.081" width="0.3048" layer="1"/>
-<wire x1="36.576" y1="13.081" x2="37.465" y2="12.192" width="0.3048" layer="16"/>
+<via x="36.83" y="13.081" extent="1-16" drill="0.5" shape="octagon"/>
+<wire x1="38.52" y1="12.7" x2="36.957" y2="12.7" width="0.3048" layer="1"/>
+<wire x1="36.957" y1="12.7" x2="36.83" y2="13.081" width="0.3048" layer="1"/>
+<wire x1="36.83" y1="13.081" x2="37.465" y2="12.192" width="0.3048" layer="16"/>
 <wire x1="37.465" y1="12.192" x2="37.465" y2="6.35" width="0.3048" layer="16"/>
-<wire x1="36.576" y1="13.081" x2="38.1" y2="14.605" width="0.3048" layer="16"/>
+<wire x1="36.83" y1="13.081" x2="38.1" y2="14.605" width="0.3048" layer="16"/>
 <wire x1="38.1" y1="14.605" x2="38.1" y2="19.05" width="0.3048" layer="16"/>
 <wire x1="38.1" y1="19.05" x2="35.56" y2="21.59" width="0.3048" layer="16"/>
@@
 <wire x1="86.36" y1="22.86" x2="84.455" y2="20.955" width="0.3048" layer="16"/>
 <wire x1="84.455" y1="20.955" x2="84.074" y2="20.955" width="0.3048" layer="16"/>
-<wire x1="57.785" y1="65.19" x2="57.785" y2="65.278" width="0.3048" layer="1"/>
-<wire x1="57.785" y1="65.278" x2="58.674" y2="66.167" width="0.3048" layer="1"/>
 <wire x1="33.715" y1="55.345" x2="32.512" y2="55.345" width="0.3048" layer="1"/>
 <wire x1="32.512" y1="55.345" x2="31.469" y2="55.345" width="0.3048" layer="1"/>
@@
 <wire x1="67.056" y1="25.4" x2="67.095" y2="25.4" width="0.3048" layer="1"/>
 <wire x1="67.056" y1="25.527" x2="67.056" y2="27.94" width="0.3048" layer="1"/>
-<wire x1="67.056" y1="27.94" x2="67.095" y2="27.94" width="0.3048" layer="1"/>
+<wire x1="67.056" y1="27.94" x2="67.095" y2="27.305" width="0.3048" layer="1"/>
 <wire x1="67.056" y1="25.527" x2="67.095" y2="25.4" width="0.3048" layer="1"/>
 <wire x1="75.057" y1="32.258" x2="76.8604" y2="32.258" width="0.3048" layer="1"/>
@@
 <wire x1="66.167" y1="28.956" x2="66.167" y2="31.115" width="0.3048" layer="1"/>
 <wire x1="67.056" y1="28.067" x2="66.167" y2="28.956" width="0.3048" layer="1"/>
-<wire x1="67.056" y1="28.067" x2="67.095" y2="27.94" width="0.3048" layer="1"/>
+<wire x1="67.056" y1="28.067" x2="67.095" y2="27.305" width="0.3048" layer="1"/>
 <wire x1="63.627" y1="18.923" x2="59.182" y2="18.923" width="0.3048" layer="1"/>
 <wire x1="66.929" y1="22.225" x2="63.627" y2="18.923" width="0.3048" layer="1"/>
@@
 <wire x1="24.638" y1="2.54" x2="23.241" y2="1.143" width="0.3048" layer="1"/>
 <wire x1="24.638" y1="2.54" x2="24.765" y2="2.54" width="0.3048" layer="1"/>
-<via x="35.306" y="52.197" extent="1-16" drill="0.4"/>
-<via x="32.512" y="54.991" extent="1-16" drill="0.4"/>
+<via x="35.306" y="52.197" extent="1-16" drill="0.5" shape="octagon"/>
+<via x="32.512" y="54.991" extent="1-16" drill="0.5" shape="octagon"/>
 <via x="76.835" y="36.449" extent="1-16" drill="0.4"/>
-<via x="56.642" y="66.04" extent="1-16" drill="0.4"/>
-<via x="55.753" y="70.231" extent="1-16" drill="0.4"/>
+<via x="56.642" y="66.04" extent="1-16" drill="0.4" shape="octagon"/>
+<via x="55.753" y="70.231" extent="1-16" drill="0.4" shape="octagon"/>
 <wire x1="27.35" y1="27.42" x2="26.555" y2="27.42" width="0.3048" layer="1"/>
 <wire x1="26.555" y1="27.42" x2="26.035" y2="27.94" width="0.3048" layer="1"/>
@@
 <wire x1="50.165" y1="59.055" x2="55.88" y2="59.055" width="0.3048" layer="1"/>
 <wire x1="55.88" y1="59.055" x2="57.15" y2="57.785" width="0.3048" layer="1"/>
-<wire x1="55.245" y1="42.545" x2="68.58" y2="29.21" width="0.3048" layer="16"/>
+<wire x1="55.245" y1="42.545" x2="68.5546" y2="28.829" width="0.3048" layer="16"/>
 <wire x1="55.245" y1="49.53" x2="55.245" y2="42.545" width="0.3048" layer="16"/>
 <wire x1="57.15" y1="51.435" x2="55.245" y2="49.53" width="0.3048" layer="1"/>
 <wire x1="57.15" y1="57.785" x2="57.15" y2="51.435" width="0.3048" layer="1"/>
-<via x="68.58" y="29.21" extent="1-16" drill="0.5" shape="octagon"/>
+<via x="68.5546" y="28.829" extent="1-16" drill="0.5" shape="octagon"/>
 <via x="55.245" y="49.53" extent="1-16" drill="0.5" shape="octagon"/>
-<wire x1="68.58" y1="29.21" x2="68.834" y2="29.464" width="0.3048" layer="1"/>
+<wire x1="68.5546" y1="28.829" x2="68.834" y2="29.464" width="0.3048" layer="1"/>
 <wire x1="68.834" y1="29.464" x2="73.8632" y2="29.464" width="0.3048" layer="1"/>
 </signal>

Commit message: switched to sparkfuns drc.
Routing:
- net GND: vias 17 -> 18
Changed lines of the file:
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@@
 <wire x1="37.465" y1="66.929" x2="37.211" y2="66.675" width="0.4064" layer="1"/>
 <wire x1="37.211" y1="66.675" x2="35.775" y2="66.675" width="0.4064" layer="1"/>
-<polygon width="0.3048" layer="16">
+<polygon width="0.3048" layer="16" isolate="0.3048">
 <vertex x="0" y="80.01"/>
 <vertex x="101.6" y="80.01"/>
@@
 <contactref element="U$8" pad="2"/>
 <contactref element="U$8" pad="4"/>
-<polygon width="0.3048" layer="1">
+<polygon width="0.3048" layer="1" isolate="0.3048">
 <vertex x="0" y="80.01"/>
 <vertex x="101.6" y="80.01"/>
@@
 <wire x1="27.35" y1="28.92" x2="28.92" y2="28.92" width="0.3048" layer="1"/>
 <wire x1="28.92" y1="28.92" x2="29.21" y2="29.21" width="0.3048" layer="1"/>
+<via x="50.165" y="71.755" extent="1-16" drill="0.5" shape="octagon"/>
+<wire x1="74.93" y1="36.615" x2="76.3524" y2="33.4518" width="0" layer="19" extent="1-1"/>
+<wire x1="75.8444" y1="23.241" x2="75.3364" y2="22.5806" width="0" layer="19" extent="1-1"/>
 <wire x1="89.115" y1="31.75" x2="89.115" y2="29.21" width="0" layer="19" extent="1-1"/>
+<wire x1="35.14" y1="12.7" x2="34.29" y2="9.74" width="0" layer="19" extent="1-1"/>
+<wire x1="67.095" y1="30.48" x2="68.795" y2="27.305" width="0" layer="19" extent="1-1"/>
 </signal>
 <signal name="N$2">

Commit message: Fixed some design rule issues.
Parts:
- moved C43 0.64 mm to (68.6, 30.5)
Routing:
- net +3.3V: track 690.6 -> 689.4 mm
- net VDDOUT: track 29.8 -> 29.1 mm

Commit message: Some minor changes.
Other:
- board size 101.3 x 80 mm -> 101.6 x 80 mm
Changed lines of the file:
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@@
 <board>
 <plain>
-<wire x1="0" y1="0" x2="101.27" y2="0" width="0" layer="20"/>
-<wire x1="101.27" y1="0" x2="101.27" y2="80" width="0" layer="20"/>
-<wire x1="101.27" y1="80" x2="0" y2="80" width="0" layer="20"/>
-<wire x1="0" y1="80" x2="0" y2="0" width="0" layer="20"/>
+<wire x1="0" y1="0" x2="101.6" y2="0" width="0" layer="20"/>
+<wire x1="101.6" y1="0" x2="101.6" y2="80.01" width="0" layer="20"/>
+<wire x1="101.6" y1="80.01" x2="0" y2="80.01" width="0" layer="20"/>
+<wire x1="0" y1="80.01" x2="0" y2="0" width="0" layer="20"/>
 </plain>
 <attributes>
